File: atari-keyboard/atari-keyboard/_autosave-atari-keyboard.kicad_pcb (KiCad board)
At the start: 2 copper layers, 310 x 133 mm, 135 parts, among them SW1 MENU, SW10 2, SW11 0, SW12 E, SW13 [-], SW14 G, SW15 CAPS, SW16 M, SW17 RESET, SW18 3, SW19 <, SW2 1, SW20 R, SW21 [=], SW22 H, SW23 LSHIFT, SW24 [,], SW25 OPTION, SW26 4, SW27 >, SW28 T, SW29 RET, SW3 9, SW30 J, SW31 Z, SW32 [.], SW33 SELECT, SW34 5, SW35 BS, SW36 Y, SW37 CTRL, SW38 K, SW39 X, SW4 W, SW40 [/], SW41 START, SW42 6, SW43 BRK, SW44 U, SW45 A, SW46 L, SW47 C, SW48 FN, SW49 HELP, SW5 P, SW50 7, SW51 TAB, SW52 I, SW53 S, SW54 [;], SW55 V, SW56 INV, SW57 ESC, SW58 8, SW59 Q, SW6 F, SW60 O, SW61 D, SW62 [+], SW63 B, SW64 SPC, SW65 RSHIFT, SW7 MULT, SW8 N, SW9 TURBO, U1 ProMicro

Commit message: Added arrow keys and joystick support.  Writing code to auto-calc key placement.
Parts:
- removed the D17 at (120.9, 9.64)
- removed the D25 at (127.6, 9.64)
- removed the D33 at (134.3, 9.64)
- removed the D41 at (141.0, 9.64)
- removed the D43 at (278.6, 38.1)
- removed the D49 at (147.7, 9.64)
- removed the D56 at (278.6, 95.2)
- removed the D9 at (114.2, 9.64)
- removed the SW25 at (195.3, 0.00)
- removed the SW33 at (219.1, 0.00)
- removed the SW35 at (252.4, 28.6)
- removed the SW41 at (242.9, 0.00)
- removed the SW43 at (271.5, 28.6)
- removed the SW49 at (266.7, 0.00)
- added D18: UP, Diode_THT:D_A-405_P7.62mm_Horizontal, B.Cu at (278.5, 95.2)
- added D2: TURBO, Diode_THT:D_A-405_P7.62mm_Horizontal, B.Cu at (59.5, 9.52)
- added D24: BRK, Diode_THT:D_A-405_P7.62mm_Horizontal, B.Cu at (273.8, 9.54)
- added D27: DOWN, Diode_THT:D_A-405_P7.62mm_Horizontal, B.Cu at (278.5, 113.8)
- added D3: RESET, Diode_THT:D_A-405_P7.62mm_Horizontal, B.Cu at (9.52, 9.52)
- added D36: LEFT, Diode_THT:D_A-405_P7.62mm_Horizontal, B.Cu at (259.4, 113.8)
- added D4: OPTION, Diode_THT:D_A-405_P7.62mm_Horizontal, B.Cu at (202.4, 9.52)
- added D45: RIGHT, Diode_THT:D_A-405_P7.62mm_Horizontal, B.Cu at (297.5, 113.8)
- added D5: SELECT, Diode_THT:D_A-405_P7.62mm_Horizontal, B.Cu at (178.6, 9.52)
- added D6: START, Diode_THT:D_A-405_P7.62mm_Horizontal, B.Cu at (154.8, 9.52)
- added D64: JS2_UP, Diode_THT:D_A-405_P7.62mm_Horizontal, B.Cu at (310.2, 56.0)
- added D65: JS2_TRIGGER, Diode_THT:D_A-405_P7.62mm_Horizontal, B.Cu at (371.3, 23.8)
- added D66: JS2_DOWN, Diode_THT:D_A-405_P7.62mm_Horizontal, B.Cu at (299.2, 56.0)
- added D67: JS2_LEFT, Diode_THT:D_A-405_P7.62mm_Horizontal, B.Cu at (357.0, 14.3)
- added D68: JS2_RIGHT, Diode_THT:D_A-405_P7.62mm_Horizontal, B.Cu at (321.2, 56.0)
- added D7: HELP, Diode_THT:D_A-405_P7.62mm_Horizontal, B.Cu at (226.2, 9.52)
- added D70: INV, Diode_THT:D_A-405_P7.62mm_Horizontal, B.Cu at (250.0, 9.57)
- added D73: JS1_UP, Diode_THT:D_A-405_P7.62mm_Horizontal, B.Cu at (332.1, 56.0)
- added D74: JS1_TRIGGER, Diode_THT:D_A-405_P7.62mm_Horizontal, B.Cu at (371.3, 33.3)
- added D75: JS1_DOWN, Diode_THT:D_A-405_P7.62mm_Horizontal, B.Cu at (354.1, 56.0)
- added D76: JS1_LEFT, Diode_THT:D_A-405_P7.62mm_Horizontal, B.Cu at (382.7, 38.1)
- added D77: JS1_RIGHT, Diode_THT:D_A-405_P7.62mm_Horizontal, B.Cu at (368.2, 45.4)
- added J1: Removed LEDS. Wire soldered to the board, Connector_PinSocket_2.54mm:PinSocket_1x02_P2.54mm_Vertical, F.Cu at (133.3, 4.76)
- added J2: PLAYER 1, Connector_Dsub:DSUB-9_Male_Horizontal_P2.77x2.84mm_EdgePinOffset9.90mm_Housed_MountingHolesOffset11.32mm, F.Cu at (290.4, 85.7)
- added J3: PLAYER 2, Connector_Dsub:DSUB-9_Male_Horizontal_P2.77x2.84mm_EdgePinOffset9.90mm_Housed_MountingHolesOffset11.32mm, F.Cu at (292.3, 28.0)
- added SW18: UP, Button_Switch_Keyboard:SW_Cherry_MX_1.00u_PCB, F.Cu at (271.3, 85.7)
- added SW23: BS, Button_Switch_Keyboard:SW_Cherry_MX_2.00u_PCB, F.Cu at (261.8, 28.6)
- added SW24: BRK, Button_Switch_Keyboard:SW_Cherry_MX_1.00u_PCB, F.Cu at (266.6, 0.00)
- added SW27: DOWN, Button_Switch_Keyboard:SW_Cherry_MX_1.00u_PCB, F.Cu at (271.3, 104.7)
- added SW36: LEFT, Button_Switch_Keyboard:SW_Cherry_MX_1.00u_PCB, F.Cu at (252.3, 104.7)
- added SW4: OPTION, Button_Switch_Keyboard:SW_Cherry_MX_1.00u_PCB, F.Cu at (195.2, 0.00)
- added SW45: RIGHT, Button_Switch_Keyboard:SW_Cherry_MX_1.00u_PCB, F.Cu at (290.4, 104.7)
- added SW5: SELECT, Button_Switch_Keyboard:SW_Cherry_MX_1.00u_PCB, F.Cu at (171.4, 0.00)
- added SW6: START, Button_Switch_Keyboard:SW_Cherry_MX_1.00u_PCB, F.Cu at (147.6, 0.00)
- added SW7: HELP, Button_Switch_Keyboard:SW_Cherry_MX_1.00u_PCB, F.Cu at (219.0, 0.00)
- moved SW3 169.1 mm to (2.38, 0.00)
- moved U1 111.2 mm to (114.2, 4.76)
- moved SW65 90.4 mm to (242.8, -0.03)
- moved D1 71.8 mm to (35.7, 9.52)
- moved SW2 33.4 mm to (52.4, 0.00)
- moved SW1 33.4 mm to (28.6, 0.00)
- moved D23 19.1 mm to (278.6, 38.1)
- renumbered D2 to D10, D10 to D11, D18 to D12, D26 to D13, D34 to D14, D42 to D15, D50 to D16, D58 to D17, D3 to D19, D11 to D20, D19 to D21, D27 to D22, D35 to D23, D51 to D25, D59 to D26, D4 to D28, D12 to D29, D20 to D30, D28 to D31, D36 to D32, D44 to D33, D52 to D34, D60 to D35, D5 to D37, D13 to D38, D21 to D39, D29 to D40, D37 to D41, D45 to D42, D53 to D43, D61 to D44, D6 to D46, D14 to D47, D22 to D48, D30 to D49, D38 to D50, D46 to D51, D54 to D52, D62 to D53, D8 to D54, D7 to D55, D15 to D56, D65 to D57, D31 to D58, D39 to D59, D47 to D60, D55 to D61, D63 to D62, D16 to D63, D48 to D69, D64 to D71, D24 to D72, D32 to D78, D40 to D79, D57 to D8, D23 to D9, SW2 to SW10, SW10 to SW11, SW18 to SW12, SW26 to SW13, SW34 to SW14, SW42 to SW15, SW50 to SW16, SW58 to SW17, SW3 to SW19, SW9 to SW2, SW11 to SW20, SW19 to SW21, SW27 to SW22, SW51 to SW25, SW59 to SW26, SW4 to SW28, SW12 to SW29, SW17 to SW3, SW20 to SW30, SW28 to SW31, SW36 to SW32, SW44 to SW33, SW52 to SW34, SW60 to SW35, SW5 to SW37, SW13 to SW38, SW21 to SW39, SW29 to SW40, SW37 to SW41, SW45 to SW42, SW53 to SW43, SW61 to SW44, SW6 to SW46, SW14 to SW47, SW22 to SW48, SW30 to SW49, SW38 to SW50, SW46 to SW51, SW54 to SW52, SW62 to SW53, SW8 to SW54, SW7 to SW55, SW15 to SW56, SW23 to SW57, SW31 to SW58, SW39 to SW59, SW47 to SW60, SW55 to SW61, SW63 to SW62, SW16 to SW63, SW48 to SW64, SW56 to SW65, SW64 to SW66, SW24 to SW67, SW32 to SW68, SW40 to SW69, SW57 to SW8, SW65 to SW9
Connections:
- D54 pad 1: R8 -> R6
- D57 pad 2: Net-(D23-Pad2) (its old number) -> Net-(D57-Pad2)
- D63 pad 1: R8 -> R7
- D78 pad 1: R8 -> R9
- D79 pad 1: R8 -> R9
- D9 pad 1: R7 -> R1
- D9 pad 2: Net-(D23-Pad2) (its old number) -> Net-(D9-Pad2)
- SW54 pad 2: C1 -> C9
- SW57 pad 1: Net-(D23-Pad2) (its old number) -> Net-(D57-Pad2)
- SW63 pad 2: C2 -> C9
- SW67 pad 2: C3 -> C9
- SW68 pad 2: C4 -> C6
- SW69 pad 2: C5 -> C7
- SW9 pad 1: Net-(D23-Pad2) (its old number) -> Net-(D9-Pad2)
- SW9 pad 2: C3 -> C9
- U1 pad 1: (no net) -> Net-(U1-Pad1)
- U1 pad 2: (no net) -> Net-(U1-Pad2)
- U1 pad 21: (no net) -> Net-(U1-Pad21)
- U1 pad 22: (no net) -> Net-(U1-Pad22)
- U1 pad 23: (no net) -> Net-(U1-Pad23)
- U1 pad 24: (no net) -> Net-(U1-Pad24)
- U1 pad 3: (no net) -> Net-(U1-Pad3)
- U1 pad 4: (no net) -> Net-(U1-Pad4)
Routing:
- net C5: track 606.3 -> 0.00 mm, vias 9 -> 0
- net C3: track 603.3 -> 0.00 mm, vias 12 -> 0
- net C4: track 597.5 -> 0.00 mm, vias 12 -> 0
- net C6: track 586.7 -> 0.00 mm, vias 11 -> 0
- net C7: track 583.3 -> 0.00 mm, vias 12 -> 0
- net C2: track 545.9 -> 0.00 mm, vias 13 -> 0
- net C1: track 509.6 -> 0.00 mm, vias 13 -> 0
- net R8: track 466.6 -> 0.00 mm, vias 2 -> 0
- net C8: track 442.5 -> 0.00 mm, vias 9 -> 0
- net R7: track 367.7 -> 0.00 mm, vias 1 -> 0
- net R5: track 355.2 -> 0.00 mm, vias 1 -> 0
- net R3: track 328.1 -> 0.00 mm, vias 2 -> 0
- net Net-(D23-Pad2) (its old number): track 286.7 -> 0.00 mm, vias 2 -> 0
- net R6: track 278.0 -> 0.00 mm, vias 1 -> 0
- net R4: track 224.1 -> 0.00 mm, vias 1 -> 0
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Other:
- board text removed: "PRO MICRO"
