File: atari-keyboard/atari-keyboard/_autosave-atari-keyboard.kicad_pcb (KiCad board)
At the start: 2 copper layers, 326 x 133 mm, 158 parts, among them J101 I2C DISPLAY, J2 PLAYER 1, J3 PLAYER 2, SW1 MENU, SW10 1, SW11 2, SW12 3, SW13 4, SW14 5, SW15 6, SW16 7, SW17 8, SW18 UP, SW19 9, SW2 TURBO, SW20 0, SW21 <, SW22 >, SW23 BS, SW24 BRK, SW25 TAB, SW26 Q, SW27 DOWN, SW28 W, SW29 E, SW3 RESET, SW30 R, SW31 T, SW32 Y, SW33 U, SW34 I, SW35 O, SW36 LEFT, SW37 P, SW38 [-], SW39 [=], SW4 OPTION, SW40 RET, SW41 CTRL, SW42 A, SW43 S, SW44 D, SW45 RIGHT, SW46 F, SW47 G, SW48 H, SW49 J, SW5 SELECT, SW50 K, SW51 L, SW52 [;], SW53 [+], SW54 N, SW55 MULT, SW56 CAPS, SW57 LSHIFT, SW58 Z, SW59 X, SW6 START, SW60 C, SW61 V, SW62 B, SW63 M, SW64 FN, SW65 INV, SW66 SPC, SW67 [,], SW68 [.], SW69 [/], SW7 HELP, SW8 ESC, SW9 RSHIFT, U101 Elite-C

Commit message: Updated to KiCad 6 and switched controller board to the Elite-C
Parts:
- J101: footprint Connector_PinHeader_2.54mm:PinHeader_1x05_P2.54mm_Horizontal -> Connector_PinHeader_2.54mm:PinHeader_1x04_P2.54mm_Horizontal
