File: atari-keyboard/atari-keyboard/atari-keyboard.kicad_pcb (KiCad board)
At the start: 2 copper layers, 326 x 133 mm, 158 parts, among them J101 I2C DISPLAY, J2 PLAYER 1, J3 PLAYER 2, SW1 MENU, SW10 1, SW11 2, SW12 3, SW13 4, SW14 5, SW15 6, SW16 7, SW17 8, SW18 UP, SW19 9, SW2 TURBO, SW20 0, SW21 <, SW22 >, SW23 BS, SW24 BRK, SW25 TAB, SW26 Q, SW27 DOWN, SW28 W, SW29 E, SW3 RESET, SW30 R, SW31 T, SW32 Y, SW33 U, SW34 I, SW35 O, SW36 LEFT, SW37 P, SW38 [-], SW39 [=], SW4 OPTION, SW40 RET, SW41 CTRL, SW42 A, SW43 S, SW44 D, SW45 RIGHT, SW46 F, SW47 G, SW48 H, SW49 J, SW5 SELECT, SW50 K, SW51 L, SW52 [;], SW53 [+], SW54 N, SW55 MULT, SW56 CAPS, SW57 LSHIFT, SW58 Z, SW59 X, SW6 START, SW60 C, SW61 V, SW62 B, SW63 M, SW64 FN, SW65 INV, SW66 SPC, SW67 [,], SW68 [.], SW69 [/], SW7 HELP, SW8 ESC, SW9 RSHIFT, U101 Elite-C

Commit message: Cleaned up schematic
Parts:
- D1, D10, D11, D12, D13, D14, D15, D16, D17, D18, D19, D2, D20, D21, D22, D23, D24, D25, D26, D27, D28, D29, D3, D30, D31, D32, D33, D34, D35, D36, D37, D38, D39, D4, D40, D41, D42, D43, D44, D45, D46, D47, D48, D49, D5, D50, D51, D52, D53, D54, D55, D56, D57, D58, D59, D6, D60, D61, D62, D63, D64, D66, D67, D68, D69, D7, D70, D71, D72, D73, D75, D76, D77, D78, D79, D8, D9: moved to F.Cu
- D65: value JS2_TRIGGER -> JS2_TRIG; moved to F.Cu
- D74: value JS1_TRIGGER -> JS1_TRIG; moved to F.Cu
- moved SW66 223.4 mm to (90.5, 104.8)
- moved SW1 222.2 mm to (61.9, 0.00)
- moved D1 222.2 mm to (69.0, 9.52)
- moved D2 222.2 mm to (92.9, 9.52)
- moved SW2 222.2 mm to (85.7, 0.00)
- moved D3 219.4 mm to (278.6, 9.52)
- moved SW3 219.4 mm to (271.5, 0.00)
- moved D6 217.7 mm to (126.2, 9.52)
- moved D5 217.7 mm to (150.0, 9.52)
- moved D4 217.7 mm to (173.8, 9.52)
- moved SW6 217.6 mm to (119.1, 0.00)
- moved SW5 217.6 mm to (142.9, 0.00)
- moved SW4 217.6 mm to (166.7, 0.00)
Connections:
- net /JS1_APaddle renamed /JS1_APAD
- net /JS1_BPaddle renamed /JS1_BPAD
- net /JS2_APaddle renamed /JS2_APAD
- net /JS2_BPaddle renamed /JS2_BPAD
- D46 pad 1: C9 -> R6
- D47 pad 1: C9 -> R6
- D48 pad 1: C9 -> R6
- D49 pad 1: C9 -> R6
- D50 pad 1: C9 -> R6
- D51 pad 1: C9 -> R6
- D52 pad 1: C9 -> R6
- D53 pad 1: C9 -> R6
- D54 pad 1: C9 -> R6
- D55 pad 1: C9 -> R7
- D56 pad 1: C9 -> R7
- D57 pad 1: C9 -> R7
- D58 pad 1: C9 -> R7
- D59 pad 1: C9 -> R7
- D60 pad 1: C9 -> R7
- D61 pad 1: C9 -> R7
- D62 pad 1: C9 -> R7
- D63 pad 1: C9 -> R7
- D64 pad 1: R8 -> Net-(D64-Pad1)
- D64 pad 2: /JS2_UP -> C1
- D65 pad 1: R8 -> Net-(D65-Pad1)
- D65 pad 2: /JS2_TRIGGER -> C2
- D66 pad 1: R8 -> Net-(D66-Pad1)
- D66 pad 2: /JS2_DOWN -> C3
- D67 pad 1: R8 -> Net-(D67-Pad1)
- D67 pad 2: /JS2_LEFT -> C4
- D68 pad 1: R8 -> Net-(D68-Pad1)
- D68 pad 2: /JS2_RIGHT -> C5
- D73 pad 1: R9 -> Net-(D73-Pad1)
- D73 pad 2: /JS1_UP -> C1
- D74 pad 1: R9 -> Net-(D74-Pad1)
- D74 pad 2: /JS1_TRIGGER -> C2
- D75 pad 1: R9 -> Net-(D75-Pad1)
- D75 pad 2: /JS1_DOWN -> C3
- D76 pad 1: R9 -> Net-(D76-Pad1)
- D76 pad 2: /JS1_LEFT -> C4
- D77 pad 1: R9 -> Net-(D77-Pad1)
- D77 pad 2: /JS1_RIGHT -> C5
- J2 pad 1: /JS1_UP -> Net-(D73-Pad1)
- J2 pad 2: /JS1_DOWN -> Net-(D75-Pad1)
- J2 pad 3: /JS1_LEFT -> Net-(D76-Pad1)
- J2 pad 4: /JS1_RIGHT -> Net-(D77-Pad1)
- J2 pad 6: /JS1_TRIGGER -> Net-(D74-Pad1)
- J3 pad 1: /JS2_UP -> Net-(D64-Pad1)
- J3 pad 2: /JS2_DOWN -> Net-(D66-Pad1)
- J3 pad 3: /JS2_LEFT -> Net-(D67-Pad1)
- J3 pad 4: /JS2_RIGHT -> Net-(D68-Pad1)
- J3 pad 6: /JS2_TRIGGER -> Net-(D65-Pad1)
- U101 pad 12: C9 -> R6
- U101 pad 25: C9 -> R7
Routing:
- net C6: track 525.8 -> 0.00 mm, vias 1 -> 0
- net C9: track 519.2 -> 0.00 mm, vias 1 -> 0
- net R8: track 496.2 -> 0.00 mm, vias 1 -> 0
- net C5: track 472.5 -> 0.00 mm, vias 2 -> 0
- net C7: track 462.6 -> 0.00 mm, vias 1 -> 0
- net C4: track 440.8 -> 0.00 mm
- net R3: track 432.1 -> 0.00 mm, vias 1 -> 0
- net C3: track 426.3 -> 0.00 mm
- net R9: track 410.3 -> 0.00 mm, vias 1 -> 0
- net R5: track 408.3 -> 0.00 mm
- net GND: track 401.1 -> 0.00 mm
- net C1: track 401.0 -> 0.00 mm
- net C2: track 399.0 -> 0.00 mm, vias 1 -> 0
- net C8: track 385.8 -> 0.00 mm, vias 1 -> 0
- net R1: track 314.7 -> 0.00 mm
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Other:
- rule pad_to_mask_clearance: 0.051 -> 0

Commit message: Did the new keyboard layout.
Parts:
- removed D1: MENU, Diode_THT:D_A-405_P7.62mm_Horizontal
- removed D10: 1, Diode_THT:D_A-405_P7.62mm_Horizontal
- removed D11: 2, Diode_THT:D_A-405_P7.62mm_Horizontal
- removed D12: 3, Diode_THT:D_A-405_P7.62mm_Horizontal
- removed D13: 4, Diode_THT:D_A-405_P7.62mm_Horizontal
- removed D14: 5, Diode_THT:D_A-405_P7.62mm_Horizontal
- removed D15: 6, Diode_THT:D_A-405_P7.62mm_Horizontal
- removed D16: 7, Diode_THT:D_A-405_P7.62mm_Horizontal
- removed D17: 8, Diode_THT:D_A-405_P7.62mm_Horizontal
- removed D18: UP, Diode_THT:D_A-405_P7.62mm_Horizontal
- removed D19: 9, Diode_THT:D_A-405_P7.62mm_Horizontal
- removed D2: TURBO, Diode_THT:D_A-405_P7.62mm_Horizontal
- removed D20: 0, Diode_THT:D_A-405_P7.62mm_Horizontal
- removed D21: <, Diode_THT:D_A-405_P7.62mm_Horizontal
- removed D22: >, Diode_THT:D_A-405_P7.62mm_Horizontal
- removed D23: BS, Diode_THT:D_A-405_P7.62mm_Horizontal
- removed D24: BRK, Diode_THT:D_A-405_P7.62mm_Horizontal
- removed D25: TAB, Diode_THT:D_A-405_P7.62mm_Horizontal
- removed D26: Q, Diode_THT:D_A-405_P7.62mm_Horizontal
- removed D27: DOWN, Diode_THT:D_A-405_P7.62mm_Horizontal
- removed D28: W, Diode_THT:D_A-405_P7.62mm_Horizontal
- removed D29: E, Diode_THT:D_A-405_P7.62mm_Horizontal
- removed D3: RESET, Diode_THT:D_A-405_P7.62mm_Horizontal
- removed D30: R, Diode_THT:D_A-405_P7.62mm_Horizontal
- removed D31: T, Diode_THT:D_A-405_P7.62mm_Horizontal
- removed D32: Y, Diode_THT:D_A-405_P7.62mm_Horizontal
- removed D33: U, Diode_THT:D_A-405_P7.62mm_Horizontal
- removed D34: I, Diode_THT:D_A-405_P7.62mm_Horizontal
- removed D35: O, Diode_THT:D_A-405_P7.62mm_Horizontal
- removed D36: LEFT, Diode_THT:D_A-405_P7.62mm_Horizontal
- removed D37: P, Diode_THT:D_A-405_P7.62mm_Horizontal
- removed D38: [-], Diode_THT:D_A-405_P7.62mm_Horizontal
- removed D39: [=], Diode_THT:D_A-405_P7.62mm_Horizontal
- removed D4: OPTION, Diode_THT:D_A-405_P7.62mm_Horizontal
- removed D40: RET, Diode_THT:D_A-405_P7.62mm_Horizontal
- removed D41: CTRL, Diode_THT:D_A-405_P7.62mm_Horizontal
- removed D42: A, Diode_THT:D_A-405_P7.62mm_Horizontal
- removed D43: S, Diode_THT:D_A-405_P7.62mm_Horizontal
- removed D44: D, Diode_THT:D_A-405_P7.62mm_Horizontal
- removed D45: RIGHT, Diode_THT:D_A-405_P7.62mm_Horizontal
- removed D46: F, Diode_THT:D_A-405_P7.62mm_Horizontal
- removed D47: G, Diode_THT:D_A-405_P7.62mm_Horizontal
- removed D48: H, Diode_THT:D_A-405_P7.62mm_Horizontal
- removed D49: J, Diode_THT:D_A-405_P7.62mm_Horizontal
- removed D5: SELECT, Diode_THT:D_A-405_P7.62mm_Horizontal
- removed D50: K, Diode_THT:D_A-405_P7.62mm_Horizontal
- removed D51: L, Diode_THT:D_A-405_P7.62mm_Horizontal
- removed D52: [;], Diode_THT:D_A-405_P7.62mm_Horizontal
- removed D53: [+], Diode_THT:D_A-405_P7.62mm_Horizontal
- removed D54: N, Diode_THT:D_A-405_P7.62mm_Horizontal
- removed D55: MULT, Diode_THT:D_A-405_P7.62mm_Horizontal
- removed D56: CAPS, Diode_THT:D_A-405_P7.62mm_Horizontal
- removed D57, D9: LSHIFT, Diode_THT:D_A-405_P7.62mm_Horizontal
- removed D58: Z, Diode_THT:D_A-405_P7.62mm_Horizontal
- removed D59: X, Diode_THT:D_A-405_P7.62mm_Horizontal
- removed D6: START, Diode_THT:D_A-405_P7.62mm_Horizontal
- removed D60: C, Diode_THT:D_A-405_P7.62mm_Horizontal
- removed D61: V, Diode_THT:D_A-405_P7.62mm_Horizontal
- removed D62: B, Diode_THT:D_A-405_P7.62mm_Horizontal
- removed D63: M, Diode_THT:D_A-405_P7.62mm_Horizontal
- removed D64: JS2_UP, Diode_THT:D_A-405_P7.62mm_Horizontal
- removed D65: JS2_TRIG, Diode_THT:D_A-405_P7.62mm_Horizontal
- removed D66: JS2_DOWN, Diode_THT:D_A-405_P7.62mm_Horizontal
- removed D67: JS2_LEFT, Diode_THT:D_A-405_P7.62mm_Horizontal
- removed D68: JS2_RIGHT, Diode_THT:D_A-405_P7.62mm_Horizontal
- removed D69: FN, Diode_THT:D_A-405_P7.62mm_Horizontal
- removed D7: HELP, Diode_THT:D_A-405_P7.62mm_Horizontal
- removed D70: INV, Diode_THT:D_A-405_P7.62mm_Horizontal
- removed D71: SPC, Diode_THT:D_A-405_P7.62mm_Horizontal
- removed D72: [,], Diode_THT:D_A-405_P7.62mm_Horizontal
- removed D73: JS1_UP, Diode_THT:D_A-405_P7.62mm_Horizontal
- removed D74: JS1_TRIG, Diode_THT:D_A-405_P7.62mm_Horizontal
- removed D75: JS1_DOWN, Diode_THT:D_A-405_P7.62mm_Horizontal
- removed D76: JS1_LEFT, Diode_THT:D_A-405_P7.62mm_Horizontal
- removed D77: JS1_RIGHT, Diode_THT:D_A-405_P7.62mm_Horizontal
- removed D78: [.], Diode_THT:D_A-405_P7.62mm_Horizontal
- removed D79: [/], Diode_THT:D_A-405_P7.62mm_Horizontal
- removed D8: ESC, Diode_THT:D_A-405_P7.62mm_Horizontal
- removed H1, H2, H3, H4: MountingHole, MountingHole:MountingHole_3.2mm_M3
- removed J2: PLAYER 1, Connector_Dsub:DSUB-9_Male_Horizontal_P2.77x2.84mm_EdgePinOffset9.90mm_Housed_MountingHolesOffset11.32mm
- removed J3: PLAYER 2, Connector_Dsub:DSUB-9_Male_Horizontal_P2.77x2.84mm_EdgePinOffset9.90mm_Housed_MountingHolesOffset11.32mm
- removed SW1: MENU, Button_Switch_Keyboard:SW_Cherry_MX_1.00u_PCB
- removed SW10: 1, Button_Switch_Keyboard:SW_Cherry_MX_1.00u_PCB
- removed SW11: 2, Button_Switch_Keyboard:SW_Cherry_MX_1.00u_PCB
- removed SW12: 3, Button_Switch_Keyboard:SW_Cherry_MX_1.00u_PCB
- removed SW13: 4, Button_Switch_Keyboard:SW_Cherry_MX_1.00u_PCB
- removed SW14: 5, Button_Switch_Keyboard:SW_Cherry_MX_1.00u_PCB
- removed SW15: 6, Button_Switch_Keyboard:SW_Cherry_MX_1.00u_PCB
- removed SW16: 7, Button_Switch_Keyboard:SW_Cherry_MX_1.00u_PCB
- removed SW17: 8, Button_Switch_Keyboard:SW_Cherry_MX_1.00u_PCB
- removed SW18: UP, Button_Switch_Keyboard:SW_Cherry_MX_1.00u_PCB
- removed SW19: 9, Button_Switch_Keyboard:SW_Cherry_MX_1.00u_PCB
- removed SW2: TURBO, Button_Switch_Keyboard:SW_Cherry_MX_1.00u_PCB
- removed SW20: 0, Button_Switch_Keyboard:SW_Cherry_MX_1.00u_PCB
- removed SW21: <, Button_Switch_Keyboard:SW_Cherry_MX_1.00u_PCB
- removed SW22: >, Button_Switch_Keyboard:SW_Cherry_MX_1.00u_PCB
- removed SW23: BS, Button_Switch_Keyboard:SW_Cherry_MX_2.00u_PCB
- removed SW24: BRK, Button_Switch_Keyboard:SW_Cherry_MX_1.00u_PCB
- removed SW25: TAB, Button_Switch_Keyboard:SW_Cherry_MX_1.75u_PCB
- removed SW26: Q, Button_Switch_Keyboard:SW_Cherry_MX_1.00u_PCB
- removed SW27: DOWN, Button_Switch_Keyboard:SW_Cherry_MX_1.00u_PCB
- removed SW28: W, Button_Switch_Keyboard:SW_Cherry_MX_1.00u_PCB
- removed SW29: E, Button_Switch_Keyboard:SW_Cherry_MX_1.00u_PCB
- removed SW3: RESET, Button_Switch_Keyboard:SW_Cherry_MX_1.00u_PCB
- removed SW30: R, Button_Switch_Keyboard:SW_Cherry_MX_1.00u_PCB
- removed SW31: T, Button_Switch_Keyboard:SW_Cherry_MX_1.00u_PCB
- removed SW32: Y, Button_Switch_Keyboard:SW_Cherry_MX_1.00u_PCB
- removed SW33: U, Button_Switch_Keyboard:SW_Cherry_MX_1.00u_PCB
- removed SW34: I, Button_Switch_Keyboard:SW_Cherry_MX_1.00u_PCB
- removed SW35: O, Button_Switch_Keyboard:SW_Cherry_MX_1.00u_PCB
- removed SW36: LEFT, Button_Switch_Keyboard:SW_Cherry_MX_1.00u_PCB
- removed SW37: P, Button_Switch_Keyboard:SW_Cherry_MX_1.00u_PCB
- removed SW38: [-], Button_Switch_Keyboard:SW_Cherry_MX_1.00u_PCB
- removed SW39: [=], Button_Switch_Keyboard:SW_Cherry_MX_1.00u_PCB
- removed SW4: OPTION, Button_Switch_Keyboard:SW_Cherry_MX_1.00u_PCB
- removed SW40: RET, Button_Switch_Keyboard:SW_Cherry_MX_1.50u_PCB
- removed SW41: CTRL, Button_Switch_Keyboard:SW_Cherry_MX_2.00u_PCB
- removed SW42: A, Button_Switch_Keyboard:SW_Cherry_MX_1.00u_PCB
- removed SW43: S, Button_Switch_Keyboard:SW_Cherry_MX_1.00u_PCB
- removed SW44: D, Button_Switch_Keyboard:SW_Cherry_MX_1.00u_PCB
- removed SW45: RIGHT, Button_Switch_Keyboard:SW_Cherry_MX_1.00u_PCB
- removed SW46: F, Button_Switch_Keyboard:SW_Cherry_MX_1.00u_PCB
- removed SW47: G, Button_Switch_Keyboard:SW_Cherry_MX_1.00u_PCB
- removed SW48: H, Button_Switch_Keyboard:SW_Cherry_MX_1.00u_PCB
- removed SW49: J, Button_Switch_Keyboard:SW_Cherry_MX_1.00u_PCB
- removed SW5: SELECT, Button_Switch_Keyboard:SW_Cherry_MX_1.00u_PCB
- removed SW50: K, Button_Switch_Keyboard:SW_Cherry_MX_1.00u_PCB
- removed SW51: L, Button_Switch_Keyboard:SW_Cherry_MX_1.00u_PCB
- removed SW52: [;], Button_Switch_Keyboard:SW_Cherry_MX_1.00u_PCB
- removed SW53: [+], Button_Switch_Keyboard:SW_Cherry_MX_1.00u_PCB
- removed SW54: N, Button_Switch_Keyboard:SW_Cherry_MX_1.00u_PCB
- removed SW55: MULT, Button_Switch_Keyboard:SW_Cherry_MX_1.00u_PCB
- removed SW56: CAPS, Button_Switch_Keyboard:SW_Cherry_MX_1.25u_PCB
- removed SW57: LSHIFT, Button_Switch_Keyboard:SW_Cherry_MX_2.25u_PCB
- removed SW58: Z, Button_Switch_Keyboard:SW_Cherry_MX_1.00u_PCB
- removed SW59: X, Button_Switch_Keyboard:SW_Cherry_MX_1.00u_PCB
- removed SW6: START, Button_Switch_Keyboard:SW_Cherry_MX_1.00u_PCB
- removed SW60: C, Button_Switch_Keyboard:SW_Cherry_MX_1.00u_PCB
- removed SW61: V, Button_Switch_Keyboard:SW_Cherry_MX_1.00u_PCB
- removed SW62: B, Button_Switch_Keyboard:SW_Cherry_MX_1.00u_PCB
- removed SW63: M, Button_Switch_Keyboard:SW_Cherry_MX_1.00u_PCB
- removed SW64: FN, Button_Switch_Keyboard:SW_Cherry_MX_1.75u_PCB
- removed SW65: INV, Button_Switch_Keyboard:SW_Cherry_MX_1.00u_PCB
- removed SW66: SPC, Button_Switch_Keyboard:SW_Cherry_MX_6.25u_PCB
- removed SW67: [,], Button_Switch_Keyboard:SW_Cherry_MX_1.00u_PCB
- removed SW68: [.], Button_Switch_Keyboard:SW_Cherry_MX_1.00u_PCB
- removed SW69: [/], Button_Switch_Keyboard:SW_Cherry_MX_1.00u_PCB
- removed SW7: HELP, Button_Switch_Keyboard:SW_Cherry_MX_1.00u_PCB
- removed SW8: ESC, Button_Switch_Keyboard:SW_Cherry_MX_1.25u_PCB
- removed SW9: RSHIFT, Button_Switch_Keyboard:SW_Cherry_MX_1.75u_PCB
- added D102: JS2_TRIG, Diode_THT:D_A-405_P7.62mm_Horizontal, F.Cu at (173.8, 66.0)
- added D103: JS2_DOWN, Diode_THT:D_A-405_P7.62mm_Horizontal, F.Cu at (135.9, 101.7)
- added D104: JS2_LEFT, Diode_THT:D_A-405_P7.62mm_Horizontal, F.Cu at (149.3, 89.5)
- added D105: JS2_RIGHT, Diode_THT:D_A-405_P7.62mm_Horizontal, F.Cu at (149.3, 93.7)
- added D106: JS1_UP, Diode_THT:D_A-405_P7.62mm_Horizontal, F.Cu at (135.9, 97.5)
- added D107: JS1_TRIG, Diode_THT:D_A-405_P7.62mm_Horizontal, F.Cu at (173.8, 61.7)
- added D108: JS1_DOWN, Diode_THT:D_A-405_P7.62mm_Horizontal, F.Cu at (113.9, 108.3)
- added D109: JS1_LEFT, Diode_THT:D_A-405_P7.62mm_Horizontal, F.Cu at (149.3, 85.2)
- added D110: JS1_RIGHT, Diode_THT:D_A-405_P7.62mm_Horizontal, F.Cu at (124.9, 108.3)
- added D111: LED, LED_THT:LED_D3.0mm, F.Cu at (143.9, 106.6)
- added D201: MENU, Diode_THT:D_A-405_P7.62mm_Horizontal, F.Cu at (142.0, 199.2)
- added D202: TURBO, Diode_THT:D_A-405_P7.62mm_Horizontal, F.Cu at (165.8, 199.2)
- added D203: RESET, Diode_THT:D_A-405_P7.62mm_Horizontal, F.Cu at (351.5, 199.2)
- added D204: OPTION, Diode_THT:D_A-405_P7.62mm_Horizontal, F.Cu at (246.7, 199.2)
- added D205: SELECT, Diode_THT:D_A-405_P7.62mm_Horizontal, F.Cu at (222.9, 199.2)
- added D206: START, Diode_THT:D_A-405_P7.62mm_Horizontal, F.Cu at (199.1, 199.2)
- added D207: HELP, Diode_THT:D_A-405_P7.62mm_Horizontal, F.Cu at (270.5, 199.2)
- added D208: ESC, Diode_THT:D_A-405_P7.62mm_Horizontal, F.Cu at (80.0, 225.4)
- added D209: RSHIFT, Diode_THT:D_A-405_P7.62mm_Horizontal, F.Cu at (322.9, 282.5)
- added D210: 1, Diode_THT:D_A-405_P7.62mm_Horizontal, F.Cu at (101.5, 225.4)
- added D211: 2, Diode_THT:D_A-405_P7.62mm_Horizontal, F.Cu at (120.5, 225.4)
- added D212: 3, Diode_THT:D_A-405_P7.62mm_Horizontal, F.Cu at (139.6, 225.4)
- added D213: 4, Diode_THT:D_A-405_P7.62mm_Horizontal, F.Cu at (158.6, 225.4)
- added D214: 5, Diode_THT:D_A-405_P7.62mm_Horizontal, F.Cu at (177.7, 225.4)
- added D215: 6, Diode_THT:D_A-405_P7.62mm_Horizontal, F.Cu at (196.7, 225.4)
- added D216: 7, Diode_THT:D_A-405_P7.62mm_Horizontal, F.Cu at (215.8, 225.4)
- added D217: 8, Diode_THT:D_A-405_P7.62mm_Horizontal, F.Cu at (234.8, 225.4)
- added D218: UP, Diode_THT:D_A-405_P7.62mm_Horizontal, F.Cu at (349.1, 282.5)
- added D219: 9, Diode_THT:D_A-405_P7.62mm_Horizontal, F.Cu at (253.9, 225.4)
- added D220: 0, Diode_THT:D_A-405_P7.62mm_Horizontal, F.Cu at (272.9, 225.4)
- added D221: <, Diode_THT:D_A-405_P7.62mm_Horizontal, F.Cu at (292.0, 225.4)
- added D222: >, Diode_THT:D_A-405_P7.62mm_Horizontal, F.Cu at (311.0, 225.4)
- added D223: BS, Diode_THT:D_A-405_P7.62mm_Horizontal, F.Cu at (339.6, 225.4)
- added D224: BRK, Diode_THT:D_A-405_P7.62mm_Horizontal, F.Cu at (327.7, 199.2)
- added D225: TAB, Diode_THT:D_A-405_P7.62mm_Horizontal, F.Cu at (84.8, 244.4)
- added D226: Q, Diode_THT:D_A-405_P7.62mm_Horizontal, F.Cu at (111.0, 244.4)
- added D227: DOWN, Diode_THT:D_A-405_P7.62mm_Horizontal, F.Cu at (349.1, 301.6)
- added D228: W, Diode_THT:D_A-405_P7.62mm_Horizontal, F.Cu at (130.1, 244.4)
- added D229: E, Diode_THT:D_A-405_P7.62mm_Horizontal, F.Cu at (149.1, 244.4)
- added D230: R, Diode_THT:D_A-405_P7.62mm_Horizontal, F.Cu at (168.2, 244.4)
- added D231: T, Diode_THT:D_A-405_P7.62mm_Horizontal, F.Cu at (187.2, 244.4)
- added D232: Y, Diode_THT:D_A-405_P7.62mm_Horizontal, F.Cu at (206.3, 244.4)
- added D233: U, Diode_THT:D_A-405_P7.62mm_Horizontal, F.Cu at (225.3, 244.4)
- added D234: I, Diode_THT:D_A-405_P7.62mm_Horizontal, F.Cu at (244.4, 244.4)
- added D235: O, Diode_THT:D_A-405_P7.62mm_Horizontal, F.Cu at (263.4, 244.4)
- added D236: LEFT, Diode_THT:D_A-405_P7.62mm_Horizontal, F.Cu at (330.1, 301.6)
- added D237: P, Diode_THT:D_A-405_P7.62mm_Horizontal, F.Cu at (282.5, 244.4)
- added D238: [-], Diode_THT:D_A-405_P7.62mm_Horizontal, F.Cu at (301.5, 244.4)
- added D239: [=], Diode_THT:D_A-405_P7.62mm_Horizontal, F.Cu at (320.6, 244.4)
- added D240: RET, Diode_THT:D_A-405_P7.62mm_Horizontal, F.Cu at (344.4, 244.4)
- added D241: CTRL, Diode_THT:D_A-405_P7.62mm_Horizontal, F.Cu at (87.2, 263.5)
- added D242: A, Diode_THT:D_A-405_P7.62mm_Horizontal, F.Cu at (115.8, 263.5)
- added D243: S, Diode_THT:D_A-405_P7.62mm_Horizontal, F.Cu at (134.8, 263.5)
- added D244: D, Diode_THT:D_A-405_P7.62mm_Horizontal, F.Cu at (153.9, 263.5)
- added D245: RIGHT, Diode_THT:D_A-405_P7.62mm_Horizontal, F.Cu at (368.2, 301.6)
- added D246: F, Diode_THT:D_A-405_P7.62mm_Horizontal, F.Cu at (172.9, 263.5)
- added D247: G, Diode_THT:D_A-405_P7.62mm_Horizontal, F.Cu at (192.0, 263.5)
- added D248: H, Diode_THT:D_A-405_P7.62mm_Horizontal, F.Cu at (211.0, 263.5)
- added D249: J, Diode_THT:D_A-405_P7.62mm_Horizontal, F.Cu at (230.1, 263.5)
- added D250: K, Diode_THT:D_A-405_P7.62mm_Horizontal, F.Cu at (249.1, 263.5)
- added D251: L, Diode_THT:D_A-405_P7.62mm_Horizontal, F.Cu at (268.2, 263.5)
- added D252: [;], Diode_THT:D_A-405_P7.62mm_Horizontal, F.Cu at (287.2, 263.5)
- added D253: [+], Diode_THT:D_A-405_P7.62mm_Horizontal, F.Cu at (306.3, 263.5)
- added D254: N, Diode_THT:D_A-405_P7.62mm_Horizontal, F.Cu at (220.5, 282.5)
- added D255: MULT, Diode_THT:D_A-405_P7.62mm_Horizontal, F.Cu at (325.3, 263.5)
- added D256: CAPS, Diode_THT:D_A-405_P7.62mm_Horizontal, F.Cu at (346.7, 263.5)
- added D257: LSHIFT, Diode_THT:D_A-405_P7.62mm_Horizontal, F.Cu at (94.3, 282.5)
- added D258: Z, Diode_THT:D_A-405_P7.62mm_Horizontal, F.Cu at (125.3, 282.5)
- added D259: X, Diode_THT:D_A-405_P7.62mm_Horizontal, F.Cu at (144.3, 282.5)
- added D260: C, Diode_THT:D_A-405_P7.62mm_Horizontal, F.Cu at (163.4, 282.5)
- added D261: V, Diode_THT:D_A-405_P7.62mm_Horizontal, F.Cu at (182.4, 282.5)
- added D262: B, Diode_THT:D_A-405_P7.62mm_Horizontal, F.Cu at (201.5, 282.5)
- added D263: M, Diode_THT:D_A-405_P7.62mm_Horizontal, F.Cu at (239.6, 282.5)
- added D264: FN, Diode_THT:D_A-405_P7.62mm_Horizontal, F.Cu at (115.8, 301.6)
- added D265: INV, Diode_THT:D_A-405_P7.62mm_Horizontal, F.Cu at (299.1, 199.2)
- added D266: SPC, Diode_THT:D_A-405_P7.62mm_Horizontal, F.Cu at (218.2, 301.6)
- added D267: [,], Diode_THT:D_A-405_P7.62mm_Horizontal, F.Cu at (258.6, 282.5)
- added D268: [.], Diode_THT:D_A-405_P7.62mm_Horizontal, F.Cu at (277.7, 282.5)
- added D269: [/], Diode_THT:D_A-405_P7.62mm_Horizontal, F.Cu at (296.7, 282.5)
- added H101: MountingHole, MountingHole:MountingHole_3.2mm_M3, F.Cu at (187.1, 66.7)
- added H102: MountingHole, MountingHole:MountingHole_3.2mm_M3, F.Cu at (162.6, 87.1)
- added H103: MountingHole, MountingHole:MountingHole_3.2mm_M3, F.Cu at (176.1, 72.1)
- added H104: MountingHole, MountingHole:MountingHole_3.2mm_M3, F.Cu at (138.2, 107.8)
- added J102: PLAYER 1, Connector_Dsub:DSUB-9_Male_Horizontal_P2.77x2.84mm_EdgePinOffset9.90mm_Housed_MountingHolesOffset11.32mm, F.Cu at (150.1, 62.9)
- added J103: I2C DISPLAY, Connector_PinHeader_2.54mm:PinHeader_1x04_P2.54mm_Horizontal, F.Cu at (136.6, 85.4)
- added SW201: MENU, Button_Switch_Keyboard:SW_Cherry_MX_1.00u_PCB, F.Cu at (134.8, 189.7)
- added SW202: TURBO, Button_Switch_Keyboard:SW_Cherry_MX_1.00u_PCB, F.Cu at (158.6, 189.7)
- added SW203: RESET, Button_Switch_Keyboard:SW_Cherry_MX_1.00u_PCB, F.Cu at (344.4, 189.7)
- added SW204: OPTION, Button_Switch_Keyboard:SW_Cherry_MX_1.00u_PCB, F.Cu at (239.6, 189.7)
- added SW205: SELECT, Button_Switch_Keyboard:SW_Cherry_MX_1.00u_PCB, F.Cu at (215.8, 189.7)
- added SW206: START, Button_Switch_Keyboard:SW_Cherry_MX_1.00u_PCB, F.Cu at (192.0, 189.7)
- added SW207: HELP, Button_Switch_Keyboard:SW_Cherry_MX_1.00u_PCB, F.Cu at (263.4, 189.7)
- added SW208: ESC, Button_Switch_Keyboard:SW_Cherry_MX_1.25u_PCB, F.Cu at (72.9, 215.8)
- added SW209: RSHIFT, Button_Switch_Keyboard:SW_Cherry_MX_2.00u_PCB, F.Cu at (315.8, 273.0)
- added SW210: 1, Button_Switch_Keyboard:SW_Cherry_MX_1.00u_PCB, F.Cu at (94.3, 215.8)
- added SW211: 2, Button_Switch_Keyboard:SW_Cherry_MX_1.00u_PCB, F.Cu at (113.4, 215.8)
- added SW212: 3, Button_Switch_Keyboard:SW_Cherry_MX_1.00u_PCB, F.Cu at (132.4, 215.8)
- added SW213: 4, Button_Switch_Keyboard:SW_Cherry_MX_1.00u_PCB, F.Cu at (151.5, 215.8)
- added SW214: 5, Button_Switch_Keyboard:SW_Cherry_MX_1.00u_PCB, F.Cu at (170.5, 215.8)
- added SW215: 6, Button_Switch_Keyboard:SW_Cherry_MX_1.00u_PCB, F.Cu at (189.6, 215.8)
- added SW216: 7, Button_Switch_Keyboard:SW_Cherry_MX_1.00u_PCB, F.Cu at (208.6, 215.8)
- added SW217: 8, Button_Switch_Keyboard:SW_Cherry_MX_1.00u_PCB, F.Cu at (227.7, 215.8)
- added SW218: UP, Button_Switch_Keyboard:SW_Cherry_MX_1.00u_PCB, F.Cu at (342.0, 273.0)
- added SW219: 9, Button_Switch_Keyboard:SW_Cherry_MX_1.00u_PCB, F.Cu at (246.7, 215.8)
- added SW220: 0, Button_Switch_Keyboard:SW_Cherry_MX_1.00u_PCB, F.Cu at (265.8, 215.8)
- added SW221: <, Button_Switch_Keyboard:SW_Cherry_MX_1.00u_PCB, F.Cu at (284.8, 215.8)
- added SW222: >, Button_Switch_Keyboard:SW_Cherry_MX_1.00u_PCB, F.Cu at (303.9, 215.8)
- added SW223: BS, Button_Switch_Keyboard:SW_Cherry_MX_2.00u_PCB, F.Cu at (332.5, 215.8)
- added SW224: BRK, Button_Switch_Keyboard:SW_Cherry_MX_1.00u_PCB, F.Cu at (320.6, 189.7)
- added SW225: TAB, Button_Switch_Keyboard:SW_Cherry_MX_1.75u_PCB, F.Cu at (77.7, 234.9)
- added SW226: Q, Button_Switch_Keyboard:SW_Cherry_MX_1.00u_PCB, F.Cu at (103.9, 234.9)
- added SW227: DOWN, Button_Switch_Keyboard:SW_Cherry_MX_1.00u_PCB, F.Cu at (342.0, 292.1)
- added SW228: W, Button_Switch_Keyboard:SW_Cherry_MX_1.00u_PCB, F.Cu at (122.9, 234.9)
- added SW229: E, Button_Switch_Keyboard:SW_Cherry_MX_1.00u_PCB, F.Cu at (142.0, 234.9)
- added SW230: R, Button_Switch_Keyboard:SW_Cherry_MX_1.00u_PCB, F.Cu at (161.0, 234.9)
- added SW231: T, Button_Switch_Keyboard:SW_Cherry_MX_1.00u_PCB, F.Cu at (180.1, 234.9)
- added SW232: Y, Button_Switch_Keyboard:SW_Cherry_MX_1.00u_PCB, F.Cu at (199.1, 234.9)
- added SW233: U, Button_Switch_Keyboard:SW_Cherry_MX_1.00u_PCB, F.Cu at (218.2, 234.9)
- added SW234: I, Button_Switch_Keyboard:SW_Cherry_MX_1.00u_PCB, F.Cu at (237.2, 234.9)
- added SW235: O, Button_Switch_Keyboard:SW_Cherry_MX_1.00u_PCB, F.Cu at (256.3, 234.9)
- added SW236: LEFT, Button_Switch_Keyboard:SW_Cherry_MX_1.00u_PCB, F.Cu at (322.9, 292.1)
- added SW237: P, Button_Switch_Keyboard:SW_Cherry_MX_1.00u_PCB, F.Cu at (275.3, 234.9)
- added SW238: [-], Button_Switch_Keyboard:SW_Cherry_MX_1.00u_PCB, F.Cu at (294.4, 234.9)
- added SW239: [=], Button_Switch_Keyboard:SW_Cherry_MX_1.00u_PCB, F.Cu at (313.4, 234.9)
- added SW240: RET, Button_Switch_Keyboard:SW_Cherry_MX_1.50u_PCB, F.Cu at (337.2, 234.9)
- added SW241: CTRL, Button_Switch_Keyboard:SW_Cherry_MX_2.00u_PCB, F.Cu at (80.0, 253.9)
- added SW242: A, Button_Switch_Keyboard:SW_Cherry_MX_1.00u_PCB, F.Cu at (108.6, 253.9)
- added SW243: S, Button_Switch_Keyboard:SW_Cherry_MX_1.00u_PCB, F.Cu at (127.7, 253.9)
- added SW244: D, Button_Switch_Keyboard:SW_Cherry_MX_1.00u_PCB, F.Cu at (146.7, 253.9)
- added SW245: RIGHT, Button_Switch_Keyboard:SW_Cherry_MX_1.00u_PCB, F.Cu at (361.0, 292.1)
- added SW246: F, Button_Switch_Keyboard:SW_Cherry_MX_1.00u_PCB, F.Cu at (165.8, 253.9)
- added SW247: G, Button_Switch_Keyboard:SW_Cherry_MX_1.00u_PCB, F.Cu at (184.8, 253.9)
- added SW248: H, Button_Switch_Keyboard:SW_Cherry_MX_1.00u_PCB, F.Cu at (203.9, 253.9)
- added SW249: J, Button_Switch_Keyboard:SW_Cherry_MX_1.00u_PCB, F.Cu at (222.9, 253.9)
- added SW250: K, Button_Switch_Keyboard:SW_Cherry_MX_1.00u_PCB, F.Cu at (242.0, 253.9)
- added SW251: L, Button_Switch_Keyboard:SW_Cherry_MX_1.00u_PCB, F.Cu at (261.0, 253.9)
- added SW252: [;], Button_Switch_Keyboard:SW_Cherry_MX_1.00u_PCB, F.Cu at (280.1, 253.9)
- added SW253: [+], Button_Switch_Keyboard:SW_Cherry_MX_1.00u_PCB, F.Cu at (299.1, 253.9)
- added SW254: N, Button_Switch_Keyboard:SW_Cherry_MX_1.00u_PCB, F.Cu at (213.4, 273.0)
- added SW255: MULT, Button_Switch_Keyboard:SW_Cherry_MX_1.00u_PCB, F.Cu at (318.2, 253.9)
- added SW256: CAPS, Button_Switch_Keyboard:SW_Cherry_MX_1.25u_PCB, F.Cu at (339.6, 253.9)
- added SW257: LSHIFT, Button_Switch_Keyboard:SW_Cherry_MX_2.25u_PCB, F.Cu at (87.2, 273.0)
- added SW258: Z, Button_Switch_Keyboard:SW_Cherry_MX_1.00u_PCB, F.Cu at (118.2, 273.0)
- added SW259: X, Button_Switch_Keyboard:SW_Cherry_MX_1.00u_PCB, F.Cu at (137.2, 273.0)
- added SW260: C, Button_Switch_Keyboard:SW_Cherry_MX_1.00u_PCB, F.Cu at (156.2, 273.0)
- added SW261: V, Button_Switch_Keyboard:SW_Cherry_MX_1.00u_PCB, F.Cu at (175.3, 273.0)
- added SW262: B, Button_Switch_Keyboard:SW_Cherry_MX_1.00u_PCB, F.Cu at (194.3, 273.0)
- added SW263: M, Button_Switch_Keyboard:SW_Cherry_MX_1.00u_PCB, F.Cu at (232.4, 273.0)
- added SW264: FN, Button_Switch_Keyboard:SW_Cherry_MX_1.75u_PCB, F.Cu at (108.6, 292.1)
- added SW265: INV, Button_Switch_Keyboard:SW_Cherry_MX_1.00u_PCB, F.Cu at (292.0, 189.7)
- added SW266: SPC, Button_Switch_Keyboard:SW_Cherry_MX_6.25u_PCB, F.Cu at (211.0, 292.1)
- added SW267: [,], Button_Switch_Keyboard:SW_Cherry_MX_1.00u_PCB, F.Cu at (251.5, 273.0)
- added SW268: [.], Button_Switch_Keyboard:SW_Cherry_MX_1.00u_PCB, F.Cu at (270.6, 273.0)
- added SW269: [/], Button_Switch_Keyboard:SW_Cherry_MX_1.00u_PCB, F.Cu at (289.6, 273.0)
- D101: value LED -> JS2_UP; footprint LED_THT:LED_D3.0mm -> Diode_THT:D_A-405_P7.62mm_Horizontal
- J101: value I2C DISPLAY -> PLAYER 2; footprint Connector_PinHeader_2.54mm:PinHeader_1x04_P2.54mm_Horizontal -> Connector_Dsub:DSUB-9_Male_Horizontal_P2.77x2.84mm_EdgePinOffset9.90mm_Housed_MountingHolesOffset11.32mm
- moved R101 159.2 mm to (184.6, 61.2), turned to 0 degrees
- moved U101 132.5 mm to (121.2, 71.1)
- moved J101 97.4 mm to (112.2, 86.0)
- moved D101 79.0 mm to (103.0, 108.3), turned to 0 degrees
Connections:
- D101 pad 2: VCC -> C1
- J101 pad 1: GND -> Net-(D101-Pad1)
- J101 pad 2: VCC -> Net-(D103-Pad1)
- J101 pad 3: SDA -> Net-(D104-Pad1)
- J101 pad 4: SCL -> Net-(D105-Pad1)
- R101 pad 2: Net-(D101-Pad1) -> Net-(D111-Pad1)

Commit message: Front silk screen added for all keys.
Other:
- board text added: "*"
- board text added: "+"
- board text added: ","
- board text added: "-"
- board text added: "."
- board text added: "/"
- board text added: "1"
- board text added: "2"
- board text added: "263.7875 228.85"
- board text added: "3"
- board text added: "4"
- board text added: "5"
- board text added: "6"
- board text added: "7"
- board text added: "9"
- board text added: ":"
- board text added: "<"
- board text added: "="
- board text added: ">"
- board text added: "A"
- board text added: "B"
- board text added: "BREAK"
- board text added: "BS"
- board text added: "C"
- board text added: "CAPS"
- board text added: "CONTROL"
- board text added: "D"
- board text added: "E"
- board text added: "ESC"
- board text added: "F"
- board text added: "FN"
- board text added: "G"
- board text added: "H"
- board text added: "HELP"
- board text added: "I"
- board text added: "INV"
- board text added: "J"
- board text added: "K"
- board text added: "L"
- board text added: "LSHIFT"
- board text added: "M"
- board text added: "MENU"
- board text added: "N"
- board text added: "O"
- board text added: "OPTION"
- board text added: "P"
- board text added: "Q"
- board text added: "R"
- board text added: "RESET"
- board text added: "RETURN"
- board text added: "RSHIFT"
- board text added: "S"
- board text added: "SELECT"
- board text added: "START"
- board text added: "T"
- board text added: "TAB"
- board text added: "TURBO"
- board text added: "U"
- board text added: "V"
- board text added: "W"
- board text added: "X"
- board text added: "Y"
- board text added: "Z"
- board text added: "←"
- board text added: "↑"
- board text added: "→"
- board text added: "↓"
Changed lines of the file:
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@@
   (gr_line locked (start 61 177.75) (end 387 177.75) (layer "Edge.Cuts") (width 0.05))
   (gr_line locked (start 387 310.75) (end 61 310.75) (layer "Edge.Cuts") (width 0.05))
+  (gr_text "  					263.7875	228.85" (at 146.58975 219.1385) (layer "F.Cu")
+    (effects (font (size 1.5 1.5) (thickness 0.3)))
+  )
+  (gr_text "+" (at 297.125 266.95) (layer "F.SilkS")
+    (effects (font (size 1.5 1.5) (thickness 0.3)))
+  )
+  (gr_text "=" (at 311.4125 247.9) (layer "F.SilkS")
+    (effects (font (size 1.5 1.5) (thickness 0.3)))
+  )
+  (gr_text "X" (at 135.2 286) (layer "F.SilkS")
+    (effects (font (size 1.5 1.5) (thickness 0.3)))
+  )
+  (gr_text "INV" (at 289.98125 202.65625) (layer "F.SilkS")
+    (effects (font (size 1.5 1.5) (thickness 0.3)))
+  )
   (gr_text "ATARI 8BIT LAYOUT USB KEYBOARD FOR EMULATORS (VERSION 1.0)" (at 220.98 205.94224) (layer "F.SilkS")
     (effects (font (size 4 4) (thickness 0.3)))
   )
+  (gr_text "2" (at 111.3875 228.85) (layer "F.SilkS")
+    (effects (font (size 1.5 1.5) (thickness 0.3)))
+  )
+  (gr_text ":" (at 278.075 266.95) (layer "F.SilkS")
+    (effects (font (size 1.5 1.5) (thickness 0.3)))
+  )
+  (gr_text "A" (at 106.625 266.95) (layer "F.SilkS")
+    (effects (font (size 1.5 1.5) (thickness 0.3)))
+  )
+  (gr_text "R" (at 159.0125 247.9) (layer "F.SilkS")
+    (effects (font (size 1.5 1.5) (thickness 0.3)))
+  )
+  (gr_text "E" (at 139.9625 247.9) (layer "F.SilkS")
+    (effects (font (size 1.5 1.5) (thickness 0.3)))
+  )
+  (gr_text "TURBO" (at 156.63125 202.65625) (layer "F.SilkS")
+    (effects (font (size 1.5 1.5) (thickness 0.3)))
+  )
+  (gr_text "*" (at 316.175 266.95) (layer "F.SilkS")
+    (effects (font (size 1.5 1.5) (thickness 0.3)))
+  )
+  (gr_text "5" (at 168.5375 228.85) (layer "F.SilkS")
+    (effects (font (size 1.5 1.5) (thickness 0.3)))
+  )
+  (gr_text "FN" (at 106.625 305.05) (layer "F.SilkS")
+    (effects (font (size 1.5 1.5) (thickness 0.3)))
+  )
+  (gr_text "S" (at 125.675 266.95) (layer "F.SilkS")
+    (effects (font (size 1.5 1.5) (thickness 0.3)))
+  )
+  (gr_text "ESC" (at 70.90625 228.85) (layer "F.SilkS")
+    (effects (font (size 1.5 1.5) (thickness 0.3)))
+  )
+  (gr_text "," (at 249.5 286) (layer "F.SilkS")
+    (effects (font (size 1.5 1.5) (thickness 0.3)))
+  )
+  (gr_text "Q" (at 101.8625 247.9) (layer "F.SilkS")
+    (effects (font (size 1.5 1.5) (thickness 0.3)))
+  )
+  (gr_text "4" (at 149.4875 228.85) (layer "F.SilkS")
+    (effects (font (size 1.5 1.5) (thickness 0.3)))
+  )
+  (gr_text "I" (at 235.2125 247.9) (layer "F.SilkS")
+    (effects (font (size 1.5 1.5) (thickness 0.3)))
+  )
+  (gr_text "9" (at 244.7375 228.85) (layer "F.SilkS")
+    (effects (font (size 1.5 1.5) (thickness 0.3)))
+  )
+  (gr_text "3" (at 130.4375 228.85) (layer "F.SilkS")
+    (effects (font (size 1.5 1.5) (thickness 0.3)))
+  )
+  (gr_text "C" (at 154.25 286) (layer "F.SilkS")
+    (effects (font (size 1.5 1.5) (thickness 0.3)))
+  )
+  (gr_text "CAPS" (at 337.60625 266.95) (layer "F.SilkS")
+    (effects (font (size 1.5 1.5) (thickness 0.3)))
+  )
+  (gr_text "<" (at 282.8375 228.85) (layer "F.SilkS")
+    (effects (font (size 1.5 1.5) (thickness 0.3)))
+  )
+  (gr_text "Y" (at 197.1125 247.9) (layer "F.SilkS")
+    (effects (font (size 1.5 1.5) (thickness 0.3)))
+  )
+  (gr_text "1" (at 92.3375 228.85) (layer "F.SilkS")
+    (effects (font (size 1.5 1.5) (thickness 0.3)))
+  )
+  (gr_text "9" (at 225.6875 228.85) (layer "F.SilkS")
+    (effects (font (size 1.5 1.5) (thickness 0.3)))
+  )
+  (gr_text "RETURN" (at 335.225 247.9) (layer "F.SilkS")
+    (effects (font (size 1.5 1.5) (thickness 0.3)))
+  )
+  (gr_text "RESET" (at 342.36875 202.65625) (layer "F.SilkS")
+    (effects (font (size 1.5 1.5) (thickness 0.3)))
+  )
+  (gr_text "G" (at 182.825 266.95) (layer "F.SilkS")
+    (effects (font (size 1.5 1.5) (thickness 0.3)))
+  )
+  (gr_text "BREAK" (at 318.55625 202.65625) (layer "F.SilkS")
+    (effects (font (size 1.5 1.5) (thickness 0.3)))
+  )
+  (gr_text "↑" (at 339.9875 286) (layer "F.SilkS")
+    (effects (font (size 1.5 1.5) (thickness 0.3)))
+  )
+  (gr_text "M" (at 230.45 286) (layer "F.SilkS")
+    (effects (font (size 1.5 1.5) (thickness 0.3)))
+  )
+  (gr_text "CONTROL" (at 78.05 266.95) (layer "F.SilkS")
+    (effects (font (size 1.5 1.5) (thickness 0.3)))
+  )
+  (gr_text "/" (at 287.6 286) (layer "F.SilkS")
+    (effects (font (size 1.5 1.5) (thickness 0.3)))
+  )
+  (gr_text "-" (at 292.3625 247.9) (layer "F.SilkS")
+    (effects (font (size 1.5 1.5) (thickness 0.3)))
+  )
+  (gr_text "OPTION" (at 237.59375 202.65625) (layer "F.SilkS")
+    (effects (font (size 1.5 1.5) (thickness 0.3)))
+  )
+  (gr_text "Z" (at 116.15 286) (layer "F.SilkS")
+    (effects (font (size 1.5 1.5) (thickness 0.3)))
+  )
+  (gr_text "H" (at 201.875 266.95) (layer "F.SilkS")
+    (effects (font (size 1.5 1.5) (thickness 0.3)))
+  )
+  (gr_text "START" (at 189.96875 202.65625) (layer "F.SilkS")
+    (effects (font (size 1.5 1.5) (thickness 0.3)))
+  )
+  (gr_text "J" (at 220.925 266.95) (layer "F.SilkS")
+    (effects (font (size 1.5 1.5) (thickness 0.3)))
+  )
+  (gr_text "." (at 268.55 286) (layer "F.SilkS")
+    (effects (font (size 1.5 1.5) (thickness 0.3)))
+  )
+  (gr_text "BS" (at 330.4625 228.85) (layer "F.SilkS")
+    (effects (font (size 1.5 1.5) (thickness 0.3)))
+  )
+  (gr_text "TAB" (at 75.66875 247.9) (layer "F.SilkS")
+    (effects (font (size 1.5 1.5) (thickness 0.3)))
+  )
+  (gr_text "7" (at 206.6375 228.85) (layer "F.SilkS")
+    (effects (font (size 1.5 1.5) (thickness 0.3)))
+  )
+  (gr_text "SELECT" (at 213.78125 202.65625) (layer "F.SilkS")
+    (effects (font (size 1.5 1.5) (thickness 0.3)))
+  )
+  (gr_text "P" (at 273.3125 247.9) (layer "F.SilkS")
+    (effects (font (size 1.5 1.5) (thickness 0.3)))
+  )
+  (gr_text "LSHIFT" (at 85.19375 286) (layer "F.SilkS")
+    (effects (font (size 1.5 1.5) (thickness 0.3)))
+  )
+  (gr_text "B" (at 192.35 286) (layer "F.SilkS")
+    (effects (font (size 1.5 1.5) (thickness 0.3)))
+  )
+  (gr_text "K" (at 239.975 266.95) (layer "F.SilkS")
+    (effects (font (size 1.5 1.5) (thickness 0.3)))
+  )
+  (gr_text "W" (at 120.9125 247.9) (layer "F.SilkS")
+    (effects (font (size 1.5 1.5) (thickness 0.3)))
+  )
+  (gr_text "O" (at 254.2625 247.9) (layer "F.SilkS")
+    (effects (font (size 1.5 1.5) (thickness 0.3)))
+  )
+  (gr_text "RSHIFT" (at 313.79375 286) (layer "F.SilkS")
+    (effects (font (size 1.5 1.5) (thickness 0.3)))
+  )
+  (gr_text "MENU" (at 132.81875 202.65625) (layer "F.SilkS")
+    (effects (font (size 1.5 1.5) (thickness 0.3)))
+  )
+  (gr_text "F" (at 163.775 266.95) (layer "F.SilkS")
+    (effects (font (size 1.5 1.5) (thickness 0.3)))
+  )
+  (gr_text "D" (at 144.725 266.95) (layer "F.SilkS")
+    (effects (font (size 1.5 1.5) (thickness 0.3)))
+  )
+  (gr_text "←" (at 320.9375 305.05) (layer "F.SilkS")
+    (effects (font (size 1.5 1.5) (thickness 0.3)))
+  )
+  (gr_text "L" (at 259.025 266.95) (layer "F.SilkS")
+    (effects (font (size 1.5 1.5) (thickness 0.3)))
+  )
+  (gr_text "HELP" (at 261.40625 202.65625) (layer "F.SilkS")
+    (effects (font (size 1.5 1.5) (thickness 0.3)))
+  )
+  (gr_text "↓" (at 339.9875 305.05) (layer "F.SilkS")
+    (effects (font (size 1.5 1.5) (thickness 0.3)))
+  )
+  (gr_text "N" (at 211.4 286) (layer "F.SilkS")
+    (effects (font (size 1.5 1.5) (thickness 0.3)))
+  )
+  (gr_text "6" (at 187.5875 228.85) (layer "F.SilkS")
+    (effects (font (size 1.5 1.5) (thickness 0.3)))
+  )
+  (gr_text "→" (at 359.0375 305.05) (layer "F.SilkS")
+    (effects (font (size 1.5 1.5) (thickness 0.3)))
+  )
+  (gr_text "U" (at 216.1625 247.9) (layer "F.SilkS")
+    (effects (font (size 1.5 1.5) (thickness 0.3)))
+  )
+  (gr_text "V" (at 173.3 286) (layer "F.SilkS")
+    (effects (font (size 1.5 1.5) (thickness 0.3)))
+  )
+  (gr_text ">" (at 301.8875 228.85) (layer "F.SilkS")
+    (effects (font (size 1.5 1.5) (thickness 0.3)))
+  )
+  (gr_text "T" (at 178.0625 247.9) (layer "F.SilkS")
+    (effects (font (size 1.5 1.5) (thickness 0.3)))
+  )
 )

Commit message: Reran placement
Parts:
- SW209: footprint Button_Switch_Keyboard:SW_Cherry_MX_2.00u_PCB -> Button_Switch_Keyboard:SW_Cherry_MX_1.75u_PCB
- moved D101 562.0 mm to (632.9, 295.2)
- moved D110 562.0 mm to (654.9, 295.2)
- moved D111 562.0 mm to (673.8, 293.5)
- moved H102 562.0 mm to (692.5, 274.0)
- moved H104 562.0 mm to (668.2, 294.7)
- moved J101 562.0 mm to (642.2, 272.9)
- moved J102 562.0 mm to (680.1, 249.8)
- moved R101 562.0 mm to (714.5, 248.1)
- moved D102 562.0 mm to (703.8, 252.9)
- moved D103 562.0 mm to (665.9, 288.6)
- moved D104 562.0 mm to (679.3, 276.4)
- moved D105 562.0 mm to (679.3, 280.6)
- moved D106 562.0 mm to (665.9, 284.4)
- moved D107 562.0 mm to (703.8, 248.6)
- moved D108 562.0 mm to (643.9, 295.2)
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Other:
- board size 326 x 133 mm -> 307 x 128.9 mm
- board text added: "0"
- board text removed: "263.7875 228.85"
- board text removed: "ATARI 8BIT LAYOUT USB KEYBOARD FOR EMULATORS (VERSION 1.0)"

Commit message: Switched over to hybrid resisters and diodes.
Parts:
- D101, D102, D103, D104, D105, D106, D107, D108, D109, D110, D201, D202, D203, D204, D205, D206, D207, D208, D209, D210, D211, D212, D213, D214, D215, D216, D217, D218, D219, D220, D221, D222, D223, D224, D225, D226, D227, D228, D229, D230, D231, D232, D233, D234, D235, D236, D237, D238, D239, D240, D241, D242, D243, D244, D245, D246, D247, D248, D249, D250, D251, D252, D253, D254, D255, D256, D257, D258, D259, D260, D261, D262, D263, D264, D265, D266, D267, D268, D269: footprint Diode_THT:D_A-405_P7.62mm_Horizontal -> keebio:Diode-dual
- R101: footprint Resistor_THT:R_Axial_DIN0204_L3.6mm_D1.6mm_P5.08mm_Horizontal -> keebio:Resistor-Hybrid
- moved R101 614.2 mm to (114.7, 115.9)
- moved D101 603.2 mm to (43.8, 165.5)
- moved D103 603.2 mm to (76.8, 159.0)
- moved D106 603.2 mm to (76.8, 154.7)
- moved D110 603.2 mm to (65.8, 165.5)
- moved D111 603.2 mm to (84.7, 163.9)
- moved H101 603.2 mm to (127.9, 124.0)
- moved H102 603.2 mm to (103.4, 144.3)
- moved H103 603.2 mm to (117.0, 129.3)
- moved H104 603.2 mm to (79.1, 165.1)
- moved J101 603.2 mm to (53.1, 143.2)
- moved J102 603.2 mm to (91.0, 120.2)
- moved U101 603.2 mm to (62.0, 128.4)
- moved D102 603.2 mm to (114.7, 123.2)
- moved D104 603.2 mm to (90.2, 146.7)
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