File: atari-keyboard/atari-keyboard/atari-keyboard.kicad_pcb (KiCad board)
At the start: 2 copper layers, 307 x 128.9 mm, 158 parts, among them J101 PLAYER 2, J102 PLAYER 1, J103 I2C DISPLAY, SW201 MENU, SW202 TURBO, SW203 RESET, SW204 OPTION, SW205 SELECT, SW206 START, SW207 HELP, SW208 ESC, SW209 RSHIFT, SW210 1, SW211 2, SW212 3, SW213 4, SW214 5, SW215 6, SW216 7, SW217 8, SW218 UP, SW219 9, SW220 0, SW221 <, SW222 >, SW223 BS, SW224 BRK, SW225 TAB, SW226 Q, SW227 DOWN, SW228 W, SW229 E, SW230 R, SW231 T, SW232 Y, SW233 U, SW234 I, SW235 O, SW236 LEFT, SW237 P, SW238 [-], SW239 [=], SW240 RET, SW241 CTRL, SW242 A, SW243 S, SW244 D, SW245 RIGHT, SW246 F, SW247 G, SW248 H, SW249 J, SW250 K, SW251 L, SW252 [;], SW253 [+], SW254 N, SW255 MULT, SW256 CAPS, SW257 LSHIFT, SW258 Z, SW259 X, SW260 C, SW261 V, SW262 B, SW263 M, SW264 FN, SW265 INV, SW266 SPC, SW267 [,], SW268 [.], SW269 [/], U101 Elite-C

Commit message: Added "POWER" button
Parts:
- added D270: POWER, keebio:Diode-dual, F.Cu at (-106.4, 173.3)
- added SW270: POWER, Button_Switch_Keyboard:SW_Cherry_MX_1.00u_PCB, F.Cu at (134.8, 189.7)
- moved D209 597.0 mm to (-271.9, 227.2), turned to 0 degrees
- moved D222 531.0 mm to (-219.9, 229.9), turned to 0 degrees
- moved D252 528.7 mm to (-240.7, 229.9), turned to 0 degrees
- moved D263 524.4 mm to (-282.3, 227.2), turned to 0 degrees
- moved D236 523.2 mm to (-188.7, 229.9), turned to 0 degrees
- moved D218 519.3 mm to (-167.9, 229.2), turned to 0 degrees
- moved D240 489.4 mm to (-140.9, 176.6), turned to 0 degrees
- moved D217 486.0 mm to (-251.1, 229.9), turned to 0 degrees
- moved D233 476.6 mm to (-251.1, 227.2), turned to 0 degrees
- moved D248 473.6 mm to (-261.5, 227.2), turned to 0 degrees
- moved D245 469.4 mm to (-75.8, 145.1), turned to 0 degrees
- moved D255 469.3 mm to (-140.9, 205.7), turned to 0 degrees
- moved D224 468.8 mm to (-140.9, 208.4), turned to 0 degrees
- moved D251 468.4 mm to (-199.1, 227.2), turned to 0 degrees
- moved D237 460.9 mm to (-178.3, 226.5), turned to 0 degrees
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Other:
- board size 307 x 128.9 mm -> 335.5 x 128.9 mm
- board text removed: "*"
- board text removed: "+"
- board text removed: ","
- board text removed: "-"
- board text removed: "."
- board text removed: "/"
- board text removed: "0"
- board text removed: "1"
- board text removed: "2"
- board text removed: "3"
- board text removed: "4"
- board text removed: "5"
- board text removed: "6"
- board text removed: "7"
- board text removed: "9"
- board text removed: ":"
- board text removed: "<"
- board text removed: "="
- board text removed: ">"
- board text removed: "A"
- board text removed: "B"
- board text removed: "BREAK"
- board text removed: "BS"
- board text removed: "C"
- board text removed: "CAPS"
- board text removed: "CONTROL"
- board text removed: "D"
- board text removed: "E"
- board text removed: "ESC"
- board text removed: "F"
- board text removed: "FN"
- board text removed: "G"
- board text removed: "H"
- board text removed: "HELP"
- board text removed: "I"
- board text removed: "INV"
- board text removed: "J"
- board text removed: "K"
- board text removed: "L"
- board text removed: "LSHIFT"
- board text removed: "M"
- board text removed: "MENU"
- board text removed: "N"
- board text removed: "O"
- board text removed: "OPTION"
- board text removed: "P"
- board text removed: "Q"
- board text removed: "R"
- board text removed: "RESET"
- board text removed: "RETURN"
- board text removed: "RSHIFT"
- board text removed: "S"
- board text removed: "SELECT"
- board text removed: "START"
- board text removed: "T"
- board text removed: "TAB"
- board text removed: "TURBO"
- board text removed: "U"
- board text removed: "V"
- board text removed: "W"
- board text removed: "X"
- board text removed: "Y"
- board text removed: "Z"
- board text removed: "←"
- board text removed: "↑"
- board text removed: "→"
- board text removed: "↓"

Commit message: Bounding box of circuit board calculated
Other:
- board size 335.5 x 128.9 mm -> 338.1 x 123.9 mm
Changed lines of the file:
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@@
     )
   )
-  (gr_rect (start 61 177.75) (end 396.4975 306.66) (layer "Edge.Cuts") (width 0.2) (fill none))
+  (gr_rect (start 120.3725 182.704) (end 144.185 206.5165) (layer "B.SilkS") (width 0.12) (fill none))
+  (gr_rect (start 58.46 182.704) (end 396.5975 306.654) (layer "Edge.Cuts") (width 0.12) (fill none))
 )

Commit message: Added mounting holes and did part layout.
Parts:
- added H201: Hole, MountingHole:MountingHole_2.2mm_M2, F.Cu at (158.5, 182.7)
- added H202: Hole, MountingHole:MountingHole_2.2mm_M2, F.Cu at (182.3, 182.7)
- added H203: Hole, MountingHole:MountingHole_2.2mm_M2, F.Cu at (372.8, 211.3)
- added H204: Hole, MountingHole:MountingHole_2.2mm_M2, F.Cu at (372.8, 235.1)
- added H205: Hole, MountingHole:MountingHole_2.2mm_M2, F.Cu at (372.8, 258.9)
- added H206: Hole, MountingHole:MountingHole_2.2mm_M2, F.Cu at (372.8, 282.7)
- added H207: Hole, MountingHole:MountingHole_2.2mm_M2, F.Cu at (372.8, 182.7)
- added H208: Hole, MountingHole:MountingHole_2.2mm_M2, F.Cu at (58.5, 211.4)
- added H209: Hole, MountingHole:MountingHole_2.2mm_M2, F.Cu at (296.6, 268.6)
- added H210: Hole, MountingHole:MountingHole_2.2mm_M2, F.Cu at (82.3, 211.4)
- added H211: Hole, MountingHole:MountingHole_2.2mm_M2, F.Cu at (101.3, 211.4)
- added H212: Hole, MountingHole:MountingHole_2.2mm_M2, F.Cu at (120.4, 211.4)
- added H213: Hole, MountingHole:MountingHole_2.2mm_M2, F.Cu at (139.4, 211.4)
- added H214: Hole, MountingHole:MountingHole_2.2mm_M2, F.Cu at (158.5, 211.4)
- added H215: Hole, MountingHole:MountingHole_2.2mm_M2, F.Cu at (177.5, 211.4)
- added H216: Hole, MountingHole:MountingHole_2.2mm_M2, F.Cu at (196.6, 211.4)
- added H217: Hole, MountingHole:MountingHole_2.2mm_M2, F.Cu at (215.6, 211.4)
- added H218: Hole, MountingHole:MountingHole_2.2mm_M2, F.Cu at (329.9, 268.6)
- added H219: Hole, MountingHole:MountingHole_2.2mm_M2, F.Cu at (234.7, 211.4)
- added H220: Hole, MountingHole:MountingHole_2.2mm_M2, F.Cu at (253.7, 211.4)
- added H221: Hole, MountingHole:MountingHole_2.2mm_M2, F.Cu at (272.8, 211.4)
- added H222: Hole, MountingHole:MountingHole_2.2mm_M2, F.Cu at (291.8, 211.4)
- added H223: Hole, MountingHole:MountingHole_2.2mm_M2, F.Cu at (310.9, 211.4)
- added H224: Hole, MountingHole:MountingHole_2.2mm_M2, F.Cu at (325.2, 182.7)
- added H225: Hole, MountingHole:MountingHole_2.2mm_M2, F.Cu at (58.5, 230.5)
- added H226: Hole, MountingHole:MountingHole_2.2mm_M2, F.Cu at (91.8, 230.5)
- added H227: Hole, MountingHole:MountingHole_2.2mm_M2, F.Cu at (329.9, 287.6)
- added H228: Hole, MountingHole:MountingHole_2.2mm_M2, F.Cu at (110.8, 230.5)
- added H229: Hole, MountingHole:MountingHole_2.2mm_M2, F.Cu at (129.9, 230.5)
- added H230: Hole, MountingHole:MountingHole_2.2mm_M2, F.Cu at (148.9, 230.5)
- added H231: Hole, MountingHole:MountingHole_2.2mm_M2, F.Cu at (168.0, 230.5)
- added H232: Hole, MountingHole:MountingHole_2.2mm_M2, F.Cu at (187.0, 230.5)
- added H233: Hole, MountingHole:MountingHole_2.2mm_M2, F.Cu at (206.1, 230.5)
- added H234: Hole, MountingHole:MountingHole_2.2mm_M2, F.Cu at (225.1, 230.5)
- added H235: Hole, MountingHole:MountingHole_2.2mm_M2, F.Cu at (244.2, 230.5)
- added H236: Hole, MountingHole:MountingHole_2.2mm_M2, F.Cu at (310.9, 287.6)
- added H237: Hole, MountingHole:MountingHole_2.2mm_M2, F.Cu at (263.2, 230.5)
- added H238: Hole, MountingHole:MountingHole_2.2mm_M2, F.Cu at (282.3, 230.5)
- added H239: Hole, MountingHole:MountingHole_2.2mm_M2, F.Cu at (301.3, 230.5)
- added H240: Hole, MountingHole:MountingHole_2.2mm_M2, F.Cu at (320.1, 230.5)
- added H241: Hole, MountingHole:MountingHole_2.2mm_M2, F.Cu at (58.5, 249.5)
- added H242: Hole, MountingHole:MountingHole_2.2mm_M2, F.Cu at (96.6, 249.5)
- added H243: Hole, MountingHole:MountingHole_2.2mm_M2, F.Cu at (115.6, 249.5)
- added H244: Hole, MountingHole:MountingHole_2.2mm_M2, F.Cu at (134.7, 249.5)
- added H245: Hole, MountingHole:MountingHole_2.2mm_M2, F.Cu at (349.0, 287.6)
- added H246: Hole, MountingHole:MountingHole_2.2mm_M2, F.Cu at (153.7, 249.5)
- added H247: Hole, MountingHole:MountingHole_2.2mm_M2, F.Cu at (172.8, 249.5)
- added H248: Hole, MountingHole:MountingHole_2.2mm_M2, F.Cu at (191.8, 249.5)
- added H249: Hole, MountingHole:MountingHole_2.2mm_M2, F.Cu at (210.9, 249.5)
- added H250: Hole, MountingHole:MountingHole_2.2mm_M2, F.Cu at (229.9, 249.5)
- added H251: Hole, MountingHole:MountingHole_2.2mm_M2, F.Cu at (249.0, 249.5)
- added H252: Hole, MountingHole:MountingHole_2.2mm_M2, F.Cu at (268.0, 249.5)
- added H253: Hole, MountingHole:MountingHole_2.2mm_M2, F.Cu at (287.1, 249.5)
- added H254: Hole, MountingHole:MountingHole_2.2mm_M2, F.Cu at (201.3, 268.6)
- added H255: Hole, MountingHole:MountingHole_2.2mm_M2, F.Cu at (306.1, 249.5)
- added H256: Hole, MountingHole:MountingHole_2.2mm_M2, F.Cu at (325.2, 249.5)
- added H257: Hole, MountingHole:MountingHole_2.2mm_M2, F.Cu at (63.2, 268.6)
- added H258: Hole, MountingHole:MountingHole_2.2mm_M2, F.Cu at (106.1, 268.6)
- added H259: Hole, MountingHole:MountingHole_2.2mm_M2, F.Cu at (125.1, 268.6)
- added H260: Hole, MountingHole:MountingHole_2.2mm_M2, F.Cu at (144.2, 268.6)
- added H261: Hole, MountingHole:MountingHole_2.2mm_M2, F.Cu at (163.2, 268.6)
- added H262: Hole, MountingHole:MountingHole_2.2mm_M2, F.Cu at (182.3, 268.6)
- added H263: Hole, MountingHole:MountingHole_2.2mm_M2, F.Cu at (220.4, 268.6)
- added H264: Hole, MountingHole:MountingHole_2.2mm_M2, F.Cu at (96.6, 287.6)
- added H265: Hole, MountingHole:MountingHole_2.2mm_M2, F.Cu at (301.3, 182.7)
- added H266: Hole, MountingHole:MountingHole_2.2mm_M2, F.Cu at (148.9, 287.6)
- added H267: Hole, MountingHole:MountingHole_2.2mm_M2, F.Cu at (239.4, 268.6)
- added H268: Hole, MountingHole:MountingHole_2.2mm_M2, F.Cu at (258.5, 268.6)
- added H269: Hole, MountingHole:MountingHole_2.2mm_M2, F.Cu at (277.5, 268.6)
- added H270: Hole, MountingHole:MountingHole_2.2mm_M2, F.Cu at (120.4, 182.7)
- moved H102 661.6 mm to (402.9, 176.3)
- moved H104 609.7 mm to (402.9, 312.9)
- moved D209 596.4 mm to (322.3, 278.5), turned to -90 degrees
- moved D206 575.8 mm to (393.7, 295.2), turned to -90 degrees
- moved D101 566.8 mm to (278.0, 196.8), turned to -90 degrees
- moved J101 550.2 mm to (268.5, 185.6), turned to 180 degrees
- moved D222 530.3 mm to (310.4, 221.4), turned to -90 degrees
- moved D252 528.1 mm to (286.6, 259.5), turned to -90 degrees
- moved D263 523.7 mm to (238.9, 278.5), turned to -90 degrees
- moved D236 522.5 mm to (329.4, 297.6), turned to -90 degrees
- moved D218 518.7 mm to (348.5, 278.5), turned to -90 degrees
- moved D103 518.1 mm to (262.9, 196.8), turned to -90 degrees
- moved D108 511.8 mm to (232.7, 196.8), turned to -90 degrees
- moved D203 503.2 mm to (393.7, 223.8), turned to -90 degrees
- moved D205 496.3 mm to (393.7, 271.4), turned to -90 degrees
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Other:
- board size 338.1 x 123.9 mm -> 358.1 x 143.9 mm
