File: atari-keyboard/atari-keyboard/atari-keyboard.kicad_pcb (KiCad board)
At the start: 2 copper layers, 355.8 x 141.4 mm, 230 parts, among them J101 PLAYER 2, J102 PLAYER 1, J103 I2C DISPLAY, SW201 MENU, SW202 TURBO, SW203 RESET, SW204 OPTION, SW205 SELECT, SW206 START, SW207 HELP, SW208 ESC, SW209 RSHIFT, SW210 1, SW211 2, SW212 3, SW213 4, SW214 5, SW215 6, SW216 7, SW217 8, SW218 UP, SW219 9, SW220 0, SW221 <, SW222 >, SW223 BS, SW224 BRK, SW225 TAB, SW226 Q, SW227 DOWN, SW228 W, SW229 E, SW230 R, SW231 T, SW232 Y, SW233 U, SW234 I, SW235 O, SW236 LEFT, SW237 P, SW238 [-], SW239 [=], SW240 RET, SW241 CTRL, SW242 A, SW243 S, SW244 D, SW245 RIGHT, SW246 F, SW247 G, SW248 H, SW249 J, SW250 K, SW251 L, SW252 [;], SW253 [+], SW254 N, SW255 MULT, SW256 CAPS, SW257 LSHIFT, SW258 Z, SW259 X, SW260 C, SW261 V, SW262 B, SW263 M, SW264 FN, SW265 INV, SW266 SPC, SW267 [,], SW268 [.], SW269 [/], SW270 POWER, U101 Elite-C

Commit message: Exclusion zones and board routed.
Parts:
- moved H201 1.50 mm to (151.3, 177.2)
- moved H202 1.50 mm to (175.1, 177.2)
- moved H203 1.50 mm to (365.6, 205.8)
- moved H204 1.50 mm to (365.6, 229.6)
- moved H205 1.50 mm to (365.6, 253.4)
- moved H206 1.50 mm to (365.6, 277.2)
- moved H207 1.50 mm to (365.6, 177.2)
- moved H208 1.50 mm to (48.9, 203.4)
- moved H209 1.50 mm to (287.1, 260.5)
- moved H210 1.50 mm to (72.7, 203.4)
- moved H211 1.50 mm to (91.8, 203.4)
- moved H212 1.50 mm to (110.8, 203.4)
- moved H213 1.50 mm to (129.9, 203.4)
- moved H214 1.50 mm to (148.9, 203.4)
- moved H215 1.50 mm to (168.0, 203.4)
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Routing:
- net C3: track 574.4 -> 518.7 mm, vias 1 -> 5
- net C4: track 534.5 -> 483.3 mm, vias 4 -> 3
- net C7: track 496.6 -> 539.5 mm, vias 5 -> 4
- net R4: track 420.8 -> 379.0 mm, vias 2 -> 0
- net R6: track 318.2 -> 291.0 mm, vias 0 -> 1
- net R2: track 394.0 -> 416.5 mm, vias 3 -> 0
- net C1: track 528.3 -> 510.3 mm
- net R8: track 392.3 -> 376.4 mm, vias 3 -> 2
- net C8: track 519.0 -> 504.0 mm, vias 4 -> 2
- net R3: track 438.9 -> 452.5 mm
- net C6: track 529.3 -> 542.0 mm
- net Net-(D101-Pad1): track 33.2 -> 21.7 mm
- net R5: track 443.3 -> 453.7 mm, vias 2 -> 3
- net R7: track 388.6 -> 378.6 mm
- net GND: track 294.0 -> 285.5 mm, vias 1 -> 0
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
Commit message: Better autogen openscad layout.  generated jlc bom&cpl
Parts:
- D218, SW218: value UP -> C_UP
- D221, SW221: value < -> LT
- D222, SW222: value > -> GT
- D227, SW227: value DOWN -> C_DOWN
- D236, SW236: value LEFT -> C_LEFT
- D238, SW238: value [-] -> DASH
- D239, SW239: value [=] -> EQUAL
- D245, SW245: value RIGHT -> C_RIGHT
- D252, SW252: value [;] -> SEMI
- D253, SW253: value [+] -> PLUS
- D255, SW255: value MULT -> ASTRIX
- D266, SW266: value SPC -> SPACE
- D267, SW267: value [,] -> COMMA
- D268, SW268: value [.] -> PERIOD
- D269, SW269: value [/] -> SLASH
- moved H240 2.00 mm to (314.9, 229.4)
Routing:
- net C7: track 539.5 -> 487.5 mm, vias 4 -> 1
- net R8: track 376.4 -> 416.2 mm, vias 2 -> 1
- net C4: track 483.3 -> 452.8 mm, vias 3 -> 2
- net C5: track 551.0 -> 524.2 mm, vias 6 -> 1
- net R2: track 416.5 -> 391.0 mm, vias 0 -> 1
- net R3: track 452.5 -> 428.7 mm, vias 1 -> 0
- net R5: track 453.7 -> 431.3 mm, vias 3 -> 2
- net C3: track 518.7 -> 500.3 mm, vias 5 -> 3
- net R4: track 379.0 -> 394.6 mm, vias 0 -> 1
- net C6: track 542.0 -> 556.9 mm, vias 2 -> 1
- net R7: track 378.6 -> 369.8 mm, vias 0 -> 1
- net R1: track 553.4 -> 562.1 mm
- net C2: track 489.8 -> 497.7 mm
- net R6: track 291.0 -> 283.6 mm
- net Net-(D103-Pad1): track 20.4 -> 27.6 mm
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
Commit message: autorouted with 1mm tracks
Parts:
- turned R101 to 180 degrees
Routing:
- net C2: track 497.7 -> 625.1 mm, vias 3 -> 4
- net R5: track 431.3 -> 530.8 mm, vias 2 -> 1
- net C6: track 556.9 -> 656.2 mm, vias 1 -> 3
- net C4: track 452.8 -> 545.6 mm, vias 2 -> 3
- net C7: track 487.5 -> 570.8 mm, vias 1 -> 5
- net R3: track 428.7 -> 490.1 mm, vias 0 -> 3
- net C1: track 508.3 -> 564.3 mm
- net C8: track 499.1 -> 539.4 mm, vias 1 -> 3
- net R1: track 562.1 -> 595.7 mm, vias 0 -> 2
- net R9: track 365.8 -> 395.3 mm, vias 0 -> 2
- net C3: track 500.3 -> 526.9 mm
- net C9: track 287.1 -> 302.9 mm
- net R2: track 391.0 -> 406.3 mm, vias 1 -> 2
- net R4: track 394.6 -> 408.2 mm
- net R7: track 369.8 -> 382.0 mm, vias 1 -> 0
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
Commit message: Reworked keyboard matrix to be a MUCH cleaner routing
Parts:
- D201: value MENU -> ESC
- D202, SW202: value TURBO -> 1
- D203, SW203: value RESET -> 2
- D204, SW204: value OPTION -> 3
- D205, SW205: value SELECT -> 4
- D206, SW206: value START -> 5
- D207, SW207: value HELP -> 6
- D208: value ESC -> 7
- D209: value RSHIFT -> 8
- D210, SW210: value 1 -> 9
- D211, SW211: value 2 -> 0
- D212, SW212: value 3 -> LT
- D213, SW213: value 4 -> GT
- D214: value 5 -> BS
- D215, SW215: value 6 -> C_UP
- D216, SW216: value 7 -> C_LEFT
- D217, SW217: value 8 -> C_DOWN
- D218, SW218: value C_UP -> C_RIGHT
- D219: value 9 -> TAB
- D220, SW220: value 0 -> Q
- D221, SW221: value LT -> W
- D222, SW222: value GT -> E
- D223: value BS -> R
- D224, SW224: value BRK -> T
- D225: value TAB -> Y
- D226, SW226: value Q -> U
- D227, SW227: value C_DOWN -> I
- D228, SW228: value W -> O
- D229, SW229: value E -> P
- D230, SW230: value R -> DASH
- D231, SW231: value T -> EQUAL
- D232: value Y -> RET
- D233, SW233: value U -> HELP
- D234, SW234: value I -> RESET
- D235, SW235: value O -> OPTION
- D236, SW236: value C_LEFT -> SELECT
- D237: value P -> CTRL
- D238, SW238: value DASH -> A
- D239, SW239: value EQUAL -> S
- D240: value RET -> D
- D241: value CTRL -> F
- D242, SW242: value A -> G
- D243, SW243: value S -> H
- D244, SW244: value D -> J
- D245, SW245: value C_RIGHT -> K
- D246, SW246: value F -> L
- D247, SW247: value G -> SEMI
- D248, SW248: value H -> PLUS
- D249, SW249: value J -> ASTRIX
- D250: value K -> CAPS
- D251, SW251: value L -> START
- D252, SW252: value SEMI -> POWER
- D253, SW253: value PLUS -> MENU
- D254, SW254: value N -> TURBO
- D255: value ASTRIX -> FN
- D256: value CAPS -> LSHIFT
- D257: value LSHIFT -> Z
- D258, SW258: value Z -> X
- D259, SW259: value X -> C
- D260, SW260: value C -> V
- D261, SW261: value V -> B
- D262, SW262: value B -> N
- D264: value FN -> COMMA
- D265, SW265: value INV -> PERIOD
- D266: value SPACE -> SLASH
- D267: value COMMA -> RSHIFT
- D268, SW268: value PERIOD -> INV
- D269, SW269: value SLASH -> BRK
- D270: value POWER -> SPACE
- SW201: value MENU -> ESC; footprint Button_Switch_Keyboard:SW_Cherry_MX_1.00u_PCB -> Button_Switch_Keyboard:SW_Cherry_MX_1.25u_PCB
- SW208: value ESC -> 7; footprint Button_Switch_Keyboard:SW_Cherry_MX_1.25u_PCB -> Button_Switch_Keyboard:SW_Cherry_MX_1.00u_PCB
- SW209: value RSHIFT -> 8; footprint Button_Switch_Keyboard:SW_Cherry_MX_1.75u_PCB -> Button_Switch_Keyboard:SW_Cherry_MX_1.00u_PCB
- SW214: value 5 -> BS; footprint Button_Switch_Keyboard:SW_Cherry_MX_1.00u_PCB -> Button_Switch_Keyboard:SW_Cherry_MX_2.00u_PCB
- SW219: value 9 -> TAB; footprint Button_Switch_Keyboard:SW_Cherry_MX_1.00u_PCB -> Button_Switch_Keyboard:SW_Cherry_MX_1.75u_PCB
- SW223: value BS -> R; footprint Button_Switch_Keyboard:SW_Cherry_MX_2.00u_PCB -> Button_Switch_Keyboard:SW_Cherry_MX_1.00u_PCB
- SW225: value TAB -> Y; footprint Button_Switch_Keyboard:SW_Cherry_MX_1.75u_PCB -> Button_Switch_Keyboard:SW_Cherry_MX_1.00u_PCB
- SW232: value Y -> RET; footprint Button_Switch_Keyboard:SW_Cherry_MX_1.00u_PCB -> Button_Switch_Keyboard:SW_Cherry_MX_1.50u_PCB
- SW237: value P -> CTRL; footprint Button_Switch_Keyboard:SW_Cherry_MX_1.00u_PCB -> Button_Switch_Keyboard:SW_Cherry_MX_2.00u_PCB
- SW240: value RET -> D; footprint Button_Switch_Keyboard:SW_Cherry_MX_1.50u_PCB -> Button_Switch_Keyboard:SW_Cherry_MX_1.00u_PCB
- SW241: value CTRL -> F; footprint Button_Switch_Keyboard:SW_Cherry_MX_2.00u_PCB -> Button_Switch_Keyboard:SW_Cherry_MX_1.00u_PCB
- SW250: value K -> CAPS; footprint Button_Switch_Keyboard:SW_Cherry_MX_1.00u_PCB -> Button_Switch_Keyboard:SW_Cherry_MX_1.25u_PCB
- SW255: value ASTRIX -> FN; footprint Button_Switch_Keyboard:SW_Cherry_MX_1.00u_PCB -> Button_Switch_Keyboard:SW_Cherry_MX_1.75u_PCB
- SW256: value CAPS -> LSHIFT; footprint Button_Switch_Keyboard:SW_Cherry_MX_1.25u_PCB -> Button_Switch_Keyboard:SW_Cherry_MX_2.00u_PCB
- SW257: value LSHIFT -> Z; footprint Button_Switch_Keyboard:SW_Cherry_MX_2.25u_PCB -> Button_Switch_Keyboard:SW_Cherry_MX_1.00u_PCB
- SW264: value FN -> COMMA; footprint Button_Switch_Keyboard:SW_Cherry_MX_1.75u_PCB -> Button_Switch_Keyboard:SW_Cherry_MX_1.00u_PCB
- SW266: value SPACE -> SLASH; footprint Button_Switch_Keyboard:SW_Cherry_MX_6.25u_PCB -> Button_Switch_Keyboard:SW_Cherry_MX_1.00u_PCB
- SW267: value COMMA -> RSHIFT; footprint Button_Switch_Keyboard:SW_Cherry_MX_1.00u_PCB -> Button_Switch_Keyboard:SW_Cherry_MX_1.75u_PCB
- SW270: value POWER -> SPACE; footprint Button_Switch_Keyboard:SW_Cherry_MX_1.00u_PCB -> Button_Switch_Keyboard:SW_Cherry_MX_6.25u_PCB
- moved D203 273.9 mm to (110.4, 211.8)
- moved H203 273.9 mm to (91.8, 203.4)
- moved SW203 273.9 mm to (103.9, 206.3)
- moved H256 260.7 mm to (56.1, 265.5)
- moved D204 256.1 mm to (129.4, 211.8)
- moved H204 256.1 mm to (110.8, 203.4)
- moved SW204 256.1 mm to (122.9, 206.3)
- moved D256 253.1 mm to (84.2, 269.0)
- moved SW256 253.1 mm to (77.7, 263.5)
- moved D205 241.0 mm to (148.5, 211.8)
- moved H205 241.0 mm to (129.9, 203.4)
- moved SW205 241.0 mm to (142.0, 206.3)
- moved D206 228.9 mm to (167.5, 211.8)
- moved H206 228.9 mm to (148.9, 203.4)
- moved SW206 228.9 mm to (161.0, 206.3)
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Connections:
- SW227 pad 2: C9 -> unconnected-(SW227-Pad2)
- SW236 pad 2: C9 -> unconnected-(SW236-Pad2)
- SW245 pad 2: C9 -> unconnected-(SW245-Pad2)
- SW254 pad 2: C9 -> unconnected-(SW254-Pad2)
- SW263 pad 2: C9 -> unconnected-(SW263-Pad2)
- SW264 pad 2: C6 -> unconnected-(SW264-Pad2)
- SW265 pad 2: C7 -> unconnected-(SW265-Pad2)
Routing:
- net C6: track 656.2 -> 0.00 mm, vias 3 -> 0
- net C2: track 625.1 -> 0.00 mm, vias 4 -> 0
- net R1: track 595.7 -> 0.00 mm, vias 2 -> 0
- net C7: track 570.8 -> 0.00 mm, vias 5 -> 0
- net C1: track 564.3 -> 0.00 mm, vias 1 -> 0
- net C4: track 545.6 -> 0.00 mm, vias 3 -> 0
- net C8: track 539.4 -> 0.00 mm, vias 3 -> 0
- net R5: track 530.8 -> 0.00 mm, vias 1 -> 0
- net C5: track 529.9 -> 0.00 mm, vias 4 -> 0
- net C3: track 526.9 -> 0.00 mm, vias 3 -> 0
- net R3: track 490.1 -> 0.00 mm, vias 3 -> 0
- net R8: track 417.4 -> 0.00 mm, vias 2 -> 0
- net R4: track 408.2 -> 0.00 mm, vias 1 -> 0
- net R2: track 406.3 -> 0.00 mm, vias 2 -> 0
- net R9: track 395.3 -> 0.00 mm, vias 2 -> 0
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
Commit message: Changed stem support type. MUCH better FDM prints.
Routing:
- net C2: track 0.00 -> 581.9 mm
- net C6: track 0.00 -> 509.3 mm
- net C7: track 0.00 -> 496.3 mm, vias 0 -> 1
- net C1: track 0.00 -> 483.3 mm, vias 0 -> 1
- net C3: track 0.00 -> 465.8 mm
- net C8: track 0.00 -> 424.5 mm
- net C4: track 0.00 -> 422.5 mm, vias 0 -> 2
- net R6: track 0.00 -> 416.5 mm
- net C5: track 0.00 -> 412.1 mm, vias 0 -> 2
- net R7: track 0.00 -> 387.2 mm, vias 0 -> 2
- net R5: track 0.00 -> 351.8 mm
- net R3: track 0.00 -> 345.8 mm
- net R1: track 0.00 -> 338.0 mm
- net R9: track 0.00 -> 331.5 mm, vias 0 -> 1
- net R4: track 0.00 -> 302.1 mm
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