File: atari-keyboard/layout-code/layout-code-py/atari-keyboard.kicad_pcb (KiCad board)
At the start: 2 copper layers, 310 x 133 mm, 156 parts, among them J1 Removed LEDS. Wire soldered t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, J2 PLAYER 1, J3 PLAYER 2, SW1 MENU, SW10 1, SW11 2, SW12 3, SW13 4, SW14 5, SW15 6, SW16 7, SW17 8, SW18 UP, SW19 9, SW2 TURBO, SW20 0, SW21 <, SW22 >, SW23 BS, SW24 BRK, SW25 TAB, SW26 Q, SW27 DOWN, SW28 W, SW29 E, SW3 RESET, SW30 R, SW31 T, SW32 Y, SW33 U, SW34 I, SW35 O, SW36 LEFT, SW37 P, SW38 [-], SW39 [=], SW4 OPTION, SW40 RET, SW41 CTRL, SW42 A, SW43 S, SW44 D, SW45 RIGHT, SW46 F, SW47 G, SW48 H, SW49 J, SW5 SELECT, SW50 K, SW51 L, SW52 [;], SW53 [+], SW54 N, SW55 MULT, SW56 CAPS, SW57 LSHIFT, SW58 Z, SW59 X, SW6 START, SW60 C, SW61 V, SW62 B, SW63 M, SW64 FN, SW65 INV, SW66 SPC, SW67 [,], SW68 [.], SW69 [/], SW7 HELP, SW8 ESC, SW9 RSHIFT, U1 ProMicro

Commit message: Have keyboard rendering in OpenSCAD almost complete.
Parts:
- D18, D27, D36, D45, D64, D65, D66, D67, D68, D73, D74, D75, D76, D77: moved to B.Cu
- D38: value [-] -> dash
- D39: value [=] -> equal
- D52, SW52: value [;] -> semi
- D53, SW53: value [+] -> plus
- D72, SW67: value [,] -> comma
- D78, SW68: value [.] -> period
- D79, SW69: value [/] -> slash
- SW38: value [-] -> minus
- SW39: value [=] -> equals
- moved J3 200.6 mm to (292.3, 28.0), turned to 90 degrees
- moved J2 196.7 mm to (290.4, 85.7), turned to 90 degrees
- moved D36 138.3 mm to (259.4, 113.8), turned to 90 degrees
- moved D27 126.9 mm to (278.5, 113.8), turned to 90 degrees
- moved SW27 118.0 mm to (271.3, 104.7)
- moved D18 117.2 mm to (278.5, 95.2), turned to 90 degrees
- moved SW18 93.2 mm to (271.3, 85.7)
- moved SW36 92.7 mm to (252.3, 104.7)
- moved SW45 90.4 mm to (290.4, 104.7)
- moved D45 73.6 mm to (297.5, 113.8), turned to 90 degrees
- moved D76 14.8 mm to (382.7, 38.1)
- moved D67 11.3 mm to (357.0, 14.3)
- moved D65 9.32 mm to (371.3, 23.8)
- moved D74 4.68 mm to (371.3, 33.3)
